File: hardware/expansion_board_V0/expansion_board_V0.brd (EAGLE design)
At the start: 160 x 100 mm, 463 parts, among them CON1 M2, CON10 QEI3, CON11 QEI2, CON2 TELEM, CON28 NC, CON3 M5, CON4 M3, CON5 M4, CON6 M0, CON7 M1, CON8 QEI1, CON9 QEI0, IC1 REF5025I, IC2 REF5030I, J1 0, J10 0, J11 0, J12 0, J13 0, J14 0, J15 0, J16 0, J19 0, J2 0, J20 nc, J21 0, J22 0, J23 0, J24 nc, J25 nc, J26 0, J27 nc, J28 nc, J29 0, J3 0, J30 0, J31 nc, J4 0, J5 0, J6 0, J7 nc, J8 0, J9 nc, Q1 25MHz, T1 MOSFET_NTR5198NL, T2 MOSFET_NTR5198NL, T3 MOSFET_NTR5198NL, U10 LAN9514, U13 LP5900_2.2, U14 ESC_TURNIGY40A, U16 ESC_CHINOI15A, U17 TPS82130, U18 TPS82130, U19 TPS82130, U2 OPA376, U20 SN74LV4052A_SO, U21 BUZZER, U4 ARDUINOR3-DIMENSION

Commit message: wip
Parts:
- moved JP7_GPIO1 401.8 mm to (270.5, -44.5)
- moved U4 390.9 mm to (307.3, -40.6)
- moved J18 385.3 mm to (298.4, -26.7)
- moved JP1_GPIO0 328.5 mm to (270.5, 16.5)
- moved L7 299.9 mm to (141.0, 106.7)
- moved L4 289.3 mm to (141.0, 111.8)
- moved L3 279.4 mm to (141.0, 109.2)
- moved L2 268.8 mm to (141.0, 114.3)
- moved CON6 237.5 mm to (106.7, 105.4), turned to 270 degrees
- moved U$23 232.4 mm to (81.3, 21.6)
- moved R44 229.6 mm to (111.8, 108.0), turned to 270 degrees
- moved C107 228.7 mm to (137.2, 106.7)
- moved C106 224.4 mm to (137.2, 109.2)
- moved C104 216.4 mm to (137.2, 111.8)
- moved C102 212.2 mm to (137.2, 114.3)
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
Commit message: wip
Parts:
- removed U$11: OSHW-LOGOS, SparkFun-Aesthetics:OSHW-LOGO-S
- moved C48 400.3 mm to (226.1, 233.7)
- moved C25 393.7 mm to (232.4, 142.2)
- moved C26 393.7 mm to (228.6, 142.2)
- moved R110 387.8 mm to (232.4, 186.7)
- moved ESC0 371.7 mm to (207.0, 147.3), turned to 90 degrees
- moved C81 364.8 mm to (199.4, 240.0)
- moved T1 360.8 mm to (195.6, 161.3)
- moved C80 360.6 mm to (199.4, 237.5)
- moved U$33 353.2 mm to (203.2, 114.3), turned to 180 degrees
- moved J10 344.7 mm to (208.3, 204.5)
- moved J9 344.7 mm to (212.1, 204.5)
- moved J6 344.4 mm to (226.1, 175.3), turned to 180 degrees
- moved C97 344.2 mm to (214.6, 176.5)
- moved J7 343.8 mm to (212.1, 240.0)
- moved J8 343.8 mm to (208.3, 240.0)
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
Commit message: wip
Parts:
- moved U$12 387.4 mm to (-40.6, 384.8)
- moved U$35 386.7 mm to (-69.8, 384.8)
- moved U2 322.4 mm to (96.5, 316.2), turned to 180 degrees
- moved J21 310.7 mm to (109.2, 330.2), turned to 90 degrees
- moved C42 287.5 mm to (114.3, 323.9), turned to 90 degrees
- moved C157 285.4 mm to (96.5, 330.2)
- moved C158 285.4 mm to (92.7, 330.2)
- moved C47 285.1 mm to (97.8, 327.7), turned to 270 degrees
- moved C46 279.7 mm to (95.2, 327.7), turned to 270 degrees
- moved C45 265.0 mm to (86.6, 319.7), turned to 90 degrees
- moved C39 255.0 mm to (111.8, 323.9), turned to 270 degrees
- moved Q1 254.5 mm to (-41.9, 355.6)
- moved R66 250.1 mm to (92.7, 316.2), turned to 270 degrees
- moved R65 248.3 mm to (92.7, 318.8), turned to 90 degrees
- moved UW2 246.9 mm to (96.5, 323.9)
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
Commit message: wip power & motor
Parts:
- moved C210 385.4 mm to (-17.7, 9.81), turned to 180 degrees
- moved C206 384.8 mm to (-19.2, 11.3), turned to 90 degrees
- moved R114 381.8 mm to (-12.9, 8.27), turned to 180 degrees
- moved C209 378.3 mm to (-17.7, 14.0), turned to 180 degrees
- moved R115 378.0 mm to (-19.2, 13.3), turned to 90 degrees
- moved C195 375.9 mm to (-17.6, 19.3), turned to 180 degrees
- moved C207 374.3 mm to (-8.87, 20.3)
- moved C208 374.2 mm to (-11.1, 20.3)
- moved R112 373.4 mm to (-17.7, 16.9)
- moved R116 373.2 mm to (-19.3, 15.4), turned to 90 degrees
- moved R118 373.0 mm to (-17.7, 12.4), turned to 180 degrees
- moved R119 372.9 mm to (-17.7, 11.1), turned to 180 degrees
- moved R113 370.8 mm to (-17.6, 18.1), turned to 180 degrees
- moved R117 369.8 mm to (-17.7, 15.3), turned to 180 degrees
- moved U20 368.0 mm to (-11.8, 14.3), turned to 180 degrees
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Other:
- board size 160 x 100 mm -> 146 x 107.6 mm

Commit message: WIP placement
Parts:
- moved C25 483.6 mm to (-189.4, -94.2), turned to 180 degrees
- moved C26 477.0 mm to (-185.6, -94.2), turned to 180 degrees
- moved U$10 473.0 mm to (-186.9, -87.9), turned to 90 degrees
- moved C87 465.7 mm to (-166.6, -113.3), turned to 180 degrees
- moved C172 451.4 mm to (-157.7, -113.3), turned to 180 degrees
- moved U$13 446.8 mm to (-157.7, -109.5), turned to 0 degrees
- moved ESC0 445.5 mm to (-164.0, -99.3), turned to 270 degrees
- moved T1 443.4 mm to (-152.6, -113.3), turned to 180 degrees
- moved U$30 430.7 mm to (-157.7, -95.5), turned to 0 degrees
- moved ESC1 418.3 mm to (-165.3, -70.1), turned to 270 degrees
- moved U$32 417.7 mm to (-160.2, -79.0), turned to 0 degrees
- moved T2 410.8 mm to (-166.6, -58.7), turned to 180 degrees
- moved U$33 405.8 mm to (-160.2, -66.3), turned to 0 degrees
- moved U14 390.7 mm to (-138.6, -87.9), turned to 180 degrees
- moved S0 385.0 mm to (50.5, -34.2), turned to 90 degrees
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Other:
- board size 146 x 107.6 mm -> 152 x 107.6 mm

Commit message: WIP placement
Parts:
- moved T2 263.2 mm to (89.5, -119.3), turned to 0 degrees
- moved C87 260.7 mm to (89.5, -64.7), turned to 0 degrees
- moved ESC1 256.4 mm to (88.3, -107.9), turned to 90 degrees
- moved ESC0 251.9 mm to (87.0, -78.7), turned to 90 degrees
- moved U$33 247.6 mm to (83.2, -111.7), turned to 180 degrees
- moved U$32 244.2 mm to (83.2, -99.0), turned to 180 degrees
- moved C25 244.0 mm to (54.4, -85.2), flipped to the bottom
- moved C172 243.2 mm to (80.7, -64.7), turned to 0 degrees
- moved U$13 241.8 mm to (80.7, -68.5), turned to 180 degrees
- moved U$10 238.9 mm to (51.9, -78.9), flipped to the bottom
- moved U$30 238.7 mm to (80.7, -82.5), turned to 180 degrees
- moved C26 236.4 mm to (50.6, -85.2), flipped to the bottom
- moved T1 233.3 mm to (75.6, -64.7), turned to 0 degrees
- moved U16 215.8 mm to (65.4, -118.0), turned to 0 degrees
- moved U14 200.2 mm to (61.6, -90.1), turned to 0 degrees
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Connections:
- net IO0: now also U$9.P$9; no longer U$9.P$1
- net IO0°: now also U$9.P$12; no longer U$9.P$20
- net IO1: now also U$9.P$8; no longer U$9.P$3
- net IO1°: now also U$9.P$13; no longer U$9.P$18
- net IO2: now also U$9.P$7; no longer U$9.P$4
- net IO2°: now also U$9.P$14; no longer U$9.P$17
- net IO3: now also U$9.P$6; no longer U$9.P$5
- net IO3°: now also U$9.P$15; no longer U$9.P$16
- net IO4: now also U$9.P$5; no longer U$9.P$6
- net IO4°: now also U$9.P$16; no longer U$9.P$15
- net IO5: now also U$9.P$4; no longer U$9.P$7
- net IO5°: now also U$9.P$17; no longer U$9.P$14
- net IO6: now also U$9.P$3; no longer U$9.P$8
- net IO6°: now also U$9.P$18; no longer U$9.P$13
- net IO7: now also U$9.P$1; no longer U$9.P$9
- net IO7°: now also U$9.P$20; no longer U$9.P$12
- net S0: now also U$8.P$9; no longer U$8.P$1
- net S0°: now also U$8.P$12; no longer U$8.P$20
- net S1: now also U$8.P$8; no longer U$8.P$3
- net S1°: now also U$8.P$13; no longer U$8.P$18
- net S2: now also U$8.P$7; no longer U$8.P$4
- net S2°: now also U$8.P$14; no longer U$8.P$17
- net S3: now also U$8.P$6; no longer U$8.P$5
- net S3°: now also U$8.P$15; no longer U$8.P$16
- net S4: now also U$8.P$5; no longer U$8.P$6
- net S4°: now also U$8.P$16; no longer U$8.P$15
- net S5: now also U$8.P$4; no longer U$8.P$7
- net S5°: now also U$8.P$17; no longer U$8.P$14
- net S6: now also U$8.P$3; no longer U$8.P$8
- net S6°: now also U$8.P$18; no longer U$8.P$13
- net S7: now also U$8.P$1; no longer U$8.P$9
- net S7°: now also U$8.P$20; no longer U$8.P$12
Routing:
- net GND: track 0.00 -> 37.5 mm
- net N$206: track 0.00 -> 27.5 mm
- net 12V: track 0.00 -> 22.5 mm
- net N$1: track 0.00 -> 5.88 mm
- net N$4: track 0.00 -> 5.87 mm
- net N$3: track 0.00 -> 5.86 mm
- net N$201: track 0.00 -> 4.25 mm
- net IO1°: track 0.00 -> 2.30 mm
- net IO5°: track 0.00 -> 2.30 mm
- net IO4°: track 0.00 -> 2.28 mm
- net IO7°: track 0.00 -> 2.27 mm
- net IO0°: track 0.00 -> 2.27 mm
- net IO3°: track 0.00 -> 2.26 mm
- net IO6°: track 0.00 -> 2.24 mm
- net N$161: track 0.00 -> 2.15 mm
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Other:
- board size 152 x 107.6 mm -> 152 x 190.6 mm

Commit message: en cours de routage. footprint wifi et arduino à revoir corrections sch  - connecteur fpga : power pins  - montage aop pour adc  - inversion pin io drivers pour faciliter le routage brd :  - inversion connecteur adc  - fixation des connecteurs fpga aux cotes nominales (à vérifier en vrai)
Parts:
- removed C103, C81: 10n, iocene:CAPC1005X55N
- removed C120, C24, C26, C82: 100n, iocene:CAPC1005X55N
- removed C177: 470u, iocene:CAPAE835X1020N
- removed R1, R2, R25, R27, R29, R3, R31, R33, R4, R51, R7, R8, R81, R91: 10k, iocene:RESC1005X40N
- removed U$5: TXS0108PWR, iocene:SOP65P640X110-20N
- removed U$6, U$7: TXB0108PWR, iocene:SOP65P640X110-20N
- removed UART0, UART1: (no value), SparkFun-Connectors:1X04_LONGPADS
- removed UART3: UART3, SparkFun-Connectors:1X04_LONGPADS
- added C137, C150: 100n, iocene:CAPC1005X55N
- added CON12: CON14, iocene:CON200P1700X400-2X7N
- added CON13: UART1, iocene:CON254P1270X400-5S
- added CON14: UART0, iocene:CON254P1270X400-5S
- added CON15: BALISE, iocene:CON254P1270X400-5S
- added J100, J101, J102, J103, J104, J105, J106, J107, J108, J109, J110, J111, J112, J113, J114, J115, J116, J117, J118, J35, J36, J37, J38, J39, J40, J41, J42, J43, J44, J45, J46, J47, J48, J49, J50, J51, J52, J53, J54, J55, J56, J57, J58, J59, J60, J61, J62, J63, J64, J65, J66, J67, J68, J69, J70, J71, J72, J73, J74, J75, J76, J77, J78, J79, J80, J81, J82, J83, J84, J85, J86, J87, J88, J89, J90, J91, J92, J93, J94, J95, J96, J97, J98, J99: JUMP_402, iocene:JUMC1005X50N
- added J119, J121, J123, J125, J127, J129, J131: nc, iocene:JUMC1005X50N
- added J120, J122, J124, J126, J128, J130, J132, J17, J32, J33, J34: 0, iocene:JUMC1005X50N
- added R11, R12, R13, R14, R15, R16: 10k, iocene:RESC1005X40N
- added U$11: TXS0108PWR, iocene:SOP65P640X110-20N
- AN0, AN1, AN2, AN3, AN4, AN5, AN6, AN7, IO0, IO1, IO2, IO3, IO4, IO5, IO6, IO7, S0, S1, S2, S3, S4, S5, S6, S7: device iocene:CON254P762X400-3N-S -> iocene:CON254P762X400-3SMT
- CON10, CON11: device iocene:CON254P1524X400-6N-S -> iocene:CON254P1270X400-5S
- J26: value 0 -> JUMP_402; device iocene:JUMC1608X50AN -> iocene:JUMC1005X50N
- J27: value nc -> JUMP_402; device iocene:JUMC1608X50AN -> iocene:JUMC1005X50N
- J30, J31: device iocene:JUMC1608X50AN -> iocene:JUMC1005X50N
- R26, R28, R30, R32, R34, R52, R67, R68, R70, R72, R74, R76, R78, R80, R90, R92: device iocene:RESC1608X50AN -> iocene:RESC1005X40N
- U$1: value OSHW-LOGOS -> TXS0108PWR; device SparkFun-Aesthetics:OSHW-LOGO-S -> iocene:SOP65P640X110-20N
- U$13, U$30, U$32, U$33: value RELAY_V23101 -> RELAY_V23101-SMT; device iocene:V23101-D0103-A201 -> iocene:V23101-D0103-A201-SMT
- U$2, U$4: value TXB0108PWR -> TXS0108PWR
- moved ESC1 316.0 mm to (-202.0, 17.0), turned to 270 degrees
- moved U$33 305.9 mm to (-197.0, 11.0), turned to 270 degrees
- moved ESC0 295.5 mm to (-202.0, -17.0), turned to 270 degrees
- moved U$32 295.5 mm to (-189.4, 15.0), turned to 90 degrees
- moved T2 288.7 mm to (-170.0, 7.10), flipped to the bottom
- moved U16 286.5 mm to (-184.5, 22.0), turned to 180 degrees
- moved U$30 283.3 mm to (-197.0, -26.0), turned to 270 degrees
- moved U$13 274.0 mm to (-189.4, -22.0), turned to 90 degrees
- moved C87 266.5 mm to (-170.2, -5.10), turned to 180 degrees
- moved U14 256.9 mm to (-183.7, -13.8), turned to 180 degrees
- moved T1 254.8 mm to (-170.0, 3.10), flipped to the bottom
- moved C22 240.2 mm to (-159.1, -5.10), flipped to the bottom, turned to 0 degrees
- moved C172 232.8 mm to (-149.5, -29.8)
- moved C206 229.8 mm to (-202.2, -135.3)
- moved R114 229.8 mm to (-195.9, -138.4)
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Connections:
- removed net /SS0: U$4.P$5
- removed net /SS1: U$4.P$9
- removed net AN10: C33.2, R53.1, UW1.38
- removed net AN11: C34.2, R55.1, UW1.37
- removed net AN12: C35.2, R57.1, UW1.36
- removed net AN13: C36.2, R60.1, UW1.35
- removed net AN14: C37.2, R62.1, UW1.34
- removed net AN15: C38.2, R64.1, UW1.33
- removed net AN8: C29.2, R47.1, UW1.40
- removed net AN9: C32.2, R49.1, UW1.39
- removed net I2C0_RST: U$5.P$4
- removed net I2C1_RST: U$5.P$7
- removed net N$108: I2C1.3, R6.1, U$5.P$15
- removed net N$109: I2C1.2, U$5.P$14
- removed net N$122: CON6.P$1, R44.P$2, U$26.P$3
- removed net N$137: CON7.P$1, R43.P$2, U$27.P$3
- removed net N$140: C136.2, CON8.3, R88.1, U$6.P$20
- removed net N$141: C203.2, CON9.2, R103.1, U$6.P$12
- removed net N$142: C204.2, CON9.3, R102.1, U$6.P$13
- removed net N$143: C197.2, R83.1, U$7.P$18
- removed net N$144: C196.2, R82.1, U$7.P$20
- removed net N$145: C199.2, R87.1, U$7.P$12
- removed net N$146: C200.2, R86.1, U$7.P$13
- removed net N$147: C201.2, R85.1, U$7.P$14
- removed net N$148: C198.2, R84.1, U$7.P$17
- removed net N$165: CON2.5, U$2.P$13
- removed net N$179: U$21.P$6
- removed net N$183: T1.P$3, U$13.11, U$30.11
- removed net N$186: J23.P$2, J25.P$2, R94.P$2, U$31.P$2
- removed net N$194: T2.P$3, U$32.11, U$33.11
- removed net N$197: J26.P$2, J27.P$2, R96.P$2, U$34.P$2
- removed net N$2: C202.2, CON8.2, R89.1, U$6.P$18
- removed net N$209: CON5.P$1, R110.P$2, U$3.P$3
- removed net N$61: U$2.P$20, UART0.3
- removed net N$64: U$2.P$17, UART1.3
- removed net N$66: U$2.P$16, UART1.2
- removed net N$67: CON2.3, U$2.P$15
- removed net N$68: CON2.2, U$2.P$14
- removed net N$69: SPI0.2, U$4.P$16
- removed net N$70: SPI0.3, U$4.P$17
- removed net N$71: SPI0.4, U$4.P$18
- removed net N$72: SPI0.5, U$4.P$20
- removed net N$73: SPI1.5, U$4.P$15
- removed net N$74: SPI1.4, U$4.P$14
- removed net N$75: SPI1.3, U$4.P$13
- removed net N$84: C88.P$2, R110.P$1, U$23.P$22, U$3.P$2
- removed net N$93: SPI1.2, U$4.P$12
- removed net N$94: I2C0.2, U$5.P$17
- removed net N$96: I2C0.3, R7.1, U$5.P$18
- removed net N$97: I2C0.4, R8.1, U$5.P$20
- removed net N$98: I2C1.4, R5.1, U$5.P$16
- removed net TELEM_PWM: U$2.P$8
- new net BALISE: J118.P$1
- new net BALISE°: CON15.5
- new net ESC_PWR: C87.+, J23.P$2, J25.P$2, R94.P$2, R96.P$2, U$31.P$3, U$34.P$2
- new net I2C0: J78.P$1, U$4.P$3
- new net I2C0°: I2C0.3, U$4.P$18
- new net I2C1: J81.P$1, U$1.P$8
- new net I2C1°: I2C1.3, U$1.P$13
- new net MISO0°: SPI0.5, U$2.P$15
- new net MISO1°: SPI1.5, U$11.P$20
- new net MOSI0°: SPI0.4, U$2.P$14
- new net MOSI1°: SPI1.4, U$11.P$18
- new net N$11: CON6.P$2, R44.P$2, U$26.P$3
- new net N$13: CON3.P$1, R110.P$2, U$3.P$3
- new net N$15: C88.P$2, CON5.P$2, U$23.P$22
- new net N$17: J17.P$2, U$24.P$5
- new net N$19: J32.P$2, U$25.P$5
- new net N$20: J33.P$2, U$20.P$5
- new net N$22: J34.P$2, U$23.P$5
- new net N$25: R65.2, R66.1, U2.P$3
- new net N$31: C13.2, J119.P$1, J120.P$1, U$2.P$19
- new net N$35: C11.2, J121.P$1, J122.P$1, R5.2, R6.2, U$4.P$19
- new net N$36: C14.2, J123.P$1, J124.P$1, R13.2, R14.2, U$1.P$19
- new net N$37: C15.2, J125.P$1, J126.P$1, U$11.P$19
- new net N$38: C16.2, J127.P$1, J128.P$1, U$8.P$19
- new net N$39: C17.2, J129.P$1, J130.P$1, U$9.P$19
- new net N$40: C19.2, J131.P$1, J132.P$1, U$10.P$19
- new net N$9: CON7.P$2, R43.P$2, U$27.P$2
- new net QEI0_A°: C203.2, CON9.2, R103.1, U$4.P$12
- new net QEI0_B°: C204.2, CON9.3, R102.1, U$4.P$13
- new net QEI1_A°: C202.2, CON8.2, R89.1, U$1.P$18
- new net QEI1_B°: C136.2, CON8.3, R88.1, U$1.P$20
- new net QEI2_A°: C199.2, R87.1, U$4.P$14
- new net QEI2_B°: C200.2, R86.1, U$4.P$15
- new net QEI2_Z°: C201.2, R85.1, U$4.P$16
- new net QEI3_A°: C198.2, R84.1, U$1.P$15
- new net QEI3_B°: C197.2, R83.1, U$1.P$16
- new net QEI3_Z°: C196.2, R82.1, U$1.P$17
- new net RX0°: CON14.2, U$2.P$18
- new net RX1°: CON13.2, U$11.P$12
- new net RX2°: CON2.2, U$2.P$16
- new net RX3: J67.P$1, U$11.P$7
- new net S0_CS: C29.2, R47.1, UW1.33
- new net S1_CS: C32.2, R49.1, UW1.34
- new net S2_CS: C33.2, R53.1, UW1.35
- new net S3_CS: C34.2, R55.1, UW1.36
- new net S4_CS: C35.2, R57.1, UW1.37
- new net S5_CS: C36.2, R60.1, UW1.38
- new net S6_CS: C37.2, R62.1, UW1.39
- new net S7_CS: C38.2, R64.1, UW1.40
- new net SCL0°: I2C0.2, R5.1, U$4.P$17
- new net SCL1°: I2C1.2, R14.1, U$1.P$12
- new net SCLK0°: SPI0.2, U$2.P$12
- new net SCLK1°: SPI1.2, U$11.P$16
- new net SDA0°: I2C0.4, R6.1, U$4.P$20
- new net SDA1°: I2C1.4, R13.1, U$1.P$14
- new net SS0: J71.P$1, U$2.P$8
- new net SS0°: SPI0.3, U$2.P$13
- new net SS1: J75.P$1, U$11.P$4
- new net SS1°: SPI1.3, U$11.P$17
- new net TELEM: J65.P$1
- new net TELEM°: CON2.5
- new net TX0°: CON14.3, U$2.P$20
- new net TX1°: CON13.3, U$11.P$13
- new net TX2°: CON2.3, U$2.P$17
- new net TX3: J66.P$1, U$11.P$6
- net 12V: now also CON15.4; no longer C177.+, C87.+, UART3.4
- net 24V: no longer J27.P$1
- net 3V3: no longer C157.2
- net 5V: now also C20.1, C22.1, CON10.5, CON11.5, CON13.4, CON14.4, J119.P$2, J121.P$2, J123.P$2, J125.P$2, J127.P$2, J129.P$2, J131.P$2; no longer C11.2, C120.2, C13.2, C15.2, C17.2, C20.2, C22.2, C24.2, C26.2, C82.2, CON10.1, CON11.1, R5.2, R6.2, R7.2, R8.2, U$10.P$19, U$2.P$19, U$4.P$19, U$5.P$19, U$6.P$19, U$7.P$19, U$8.P$19, U$9.P$19, UART0.4, UART1.4
- net A12V: no longer J26.P$1
- net A5V: now also U$30.11, U$32.11; no longer U$30.2, U$32.2
- net AD0_CLK: now also J82.P$1
- net AD0_DRDY: now also J83.P$1
- net AD0_MISO: now also J86.P$1
- net AD0_SCLK: now also J85.P$1
- net AD0_SYNC: now also J84.P$1
- net AD0_VREF: now also U$21.P$6; no longer C103.2, C81.2
- net AD1_DRDY: now also J88.P$1
- net AD1_MISO: now also J92.P$1
- net AD1_MOSI: now also J91.P$1
- net AD1_RST: now also J87.P$1
- net AD1_SCLK: now also J90.P$1
- net AD1_SS: now also J89.P$1
- net AN0: now also R67.2, UW1.45; no longer R67.P$2, UW1.4
- net AN1: now also R68.2, UW1.46; no longer R68.P$2, UW1.3
- net AN2: now also R70.2, UW1.47; no longer R70.P$2, UW1.2
- net AN3: now also R72.2, UW1.48; no longer R72.P$2, UW1.1
- net AN4: now also R74.2, UW1.1; no longer R74.P$2, UW1.48
- net AN5: now also R76.2, UW1.2; no longer R76.P$2, UW1.47
- net AN6: now also R78.2, UW1.3; no longer R78.P$2, UW1.46
- net AN7: now also R80.2, UW1.4; no longer R80.P$2, UW1.45
- net BUZZER: now also J93.P$1
- net D3V3: now also C137.2, C150.2, C157.2, J120.P$2, J122.P$2, J124.P$2, J126.P$2, J128.P$2, J130.P$2, J132.P$2, R11.2, R12.2, R15.2, R16.2, U$1.P$10, U$1.P$2, U$11.P$10, U$11.P$2; no longer C14.2, C16.2, C19.2, JP1_GPIO0.11, JP7_GPIO1.11, R1.2, R2.2, R3.2, R4.2, U$5.P$10, U$5.P$2, U$6.P$10, U$6.P$2, U$7.P$10, U$7.P$2
- net ESC0_DIR: now also J115.P$1
- net ESC0_PWM: now also J114.P$1
- net ESC1_DIR: now also J113.P$1
- net ESC1_PWM: now also J116.P$1
- net GND: now also C137.1, C150.1, C20.2, C22.2, CON10.1, CON11.1, CON13.1, CON14.1, CON15.1, U$1.P$11, U$11.P$11, U2.P$1; no longer C103.1, C120.1, C177.-, C20.1, C22.1, C24.1, C26.1, C81.1, C82.1, CON10.2, CON10.6, CON11.2, CON11.6, R25.2, R27.2, R29.2, R31.2, R33.2, R51.2, R81.2, R91.2, U$5.P$11, U$6.P$11, U$7.P$11, U2.P$3, UART0.1, UART1.1, UART3.1
- net IO0: now also J41.P$1
- net IO0°: now also R26.2; no longer R25.1, R26.P$2
- net IO1: now also J42.P$1
- net IO1°: now also R28.2; no longer R27.1, R28.P$2
- net IO2: now also J43.P$1
- net IO2°: now also R30.2; no longer R29.1, R30.P$2
- net IO3: now also J44.P$1
- net IO3°: now also R32.2; no longer R31.1, R32.P$2
- net IO4: now also J45.P$1
- net IO4°: now also R34.2; no longer R33.1, R34.P$2
- net IO5: now also J46.P$1
- net IO5°: now also R52.2; no longer R51.1, R52.P$2
- net IO6: now also J47.P$1
- net IO6°: now also R90.2; no longer R81.1, R90.P$2
- net IO7: now also J48.P$1
- net IO7°: now also R92.2; no longer R91.1, R92.P$2
- net LV_MUXA: now also J94.P$1
- net LV_MUXB: now also J95.P$1
- net M0_FAULT: now also J109.P$1
- net M0_PWMA: now also J97.P$1
- net M0_PWMB: now also J98.P$1
- net M1_FAULT: now also J110.P$1
- net M1_PWMA: now also J99.P$1
- net M1_PWMB: now also J100.P$1
- net M23_FAULT: now also J111.P$1
- net M2_PWMA: now also J101.P$1
- net M2_PWMB: now also J102.P$1
- net M3_PWMA: now also J103.P$1
- net M3_PWMB: now also J104.P$1
- net M45_FAULT: now also J112.P$1
- net M4_PWMA: now also J105.P$1
- net M4_PWMB: now also J106.P$1
- net M5_PWMA: now also J107.P$1
- net M5_PWMB: now also J108.P$1
- net MISO0: now also J68.P$1, U$2.P$6; no longer U$4.P$1
- net MISO1: now also J72.P$1, U$11.P$1; no longer U$4.P$6
- net MOSI0: now also J69.P$1, U$2.P$7; no longer U$4.P$3
- net MOSI1: now also J73.P$1, U$11.P$3; no longer U$4.P$7
- net N$114: now also J17.P$1
- net N$117: no longer U$24.P$5
- net N$126: now also CON6.P$1; no longer CON6.P$2
- net N$131: now also J32.P$1
- net N$133: no longer U$25.P$5
- net N$138: now also U$27.P$3; no longer U$27.P$2
- net N$139: now also CON7.P$1; no longer CON7.P$2
- net N$14: now also U$21.P$2; no longer U$21.P$3
- net N$156: now also R92.1; no longer R92.P$1
- net N$158: now also R26.1; no longer R26.P$1
- net N$159: now also R28.1; no longer R28.P$1
- net N$16: now also CON4.P$2; no longer CON4.P$1
- net N$160: now also R30.1; no longer R30.P$1
- net N$161: now also R32.1; no longer R32.P$1
- net N$162: now also R34.1; no longer R34.P$1
- net N$163: now also R52.1; no longer R52.P$1
- net N$164: now also R90.1; no longer R90.P$1
- net N$171: now also CON11.4; no longer CON11.3
- net N$172: now also CON11.3; no longer CON11.4
- net N$173: now also CON11.2; no longer CON11.5
- net N$174: now also CON10.4; no longer CON10.3
- net N$175: now also CON10.3; no longer CON10.4
- net N$176: now also CON10.2; no longer CON10.5
- net N$177: now also U14.W; no longer U14.V
- net N$178: now also U14.U; no longer U14.W
- net N$182: now also U14.V; no longer U14.U
- net N$185: now also U$31.P$2; no longer U$31.P$3
- net N$189: now also U16.W; no longer U16.V
- net N$190: now also U16.U; no longer U16.W
- net N$193: now also U16.V; no longer U16.U
- net N$27: now also R80.1; no longer R80.P$1
- net N$28: now also R67.1; no longer R67.P$1
- net N$30: now also R68.1; no longer R68.P$1
- net N$32: now also R70.1; no longer R70.P$1
- net N$33: now also R72.1; no longer R72.P$1
- net N$34: now also R74.1; no longer R74.P$1
- net N$5: no longer U$20.P$5
- net N$52: now also T2.P$3, U$32.2, U$33.11; no longer R65.2, R66.1, U2.P$1
- net N$55: now also CON1.P$1; no longer CON1.P$2
- net N$56: now also U$22.P$3; no longer U$22.P$2
- net N$57: now also J33.P$1
- net N$58: now also R76.1; no longer R76.P$1
- net N$59: now also R78.1; no longer R78.P$1
- net N$60: now also CON4.P$1, U$21.P$3; no longer CON4.P$2, U$21.P$2
- net N$63: now also T1.P$3, U$13.11, U$30.2; no longer U$2.P$18, UART0.2
- net N$76: now also CON1.P$2, U$22.P$2; no longer CON1.P$1, U$22.P$3
- net N$81: now also R110.P$1, U$3.P$2; no longer CON3.P$2
- net N$82: now also CON3.P$2; no longer CON3.P$1
- net N$83: now also CON5.P$1; no longer CON5.P$2
- net N$85: now also J34.P$1
- net N$88: no longer U$23.P$5
- net QEI0_A: now also J51.P$1, U$4.P$9; no longer U$6.P$8
- net QEI0_B: now also J52.P$1, U$4.P$8; no longer U$6.P$9
- net QEI1_A: now also J49.P$1, U$1.P$3; no longer U$6.P$1
- net QEI1_B: now also J50.P$1, U$1.P$1; no longer U$6.P$3
- net QEI2_A: now also J56.P$1, U$4.P$7; no longer U$7.P$7
- net QEI2_B: now also J57.P$1, U$4.P$6; no longer U$7.P$8
- net QEI2_Z: now also J58.P$1, U$4.P$5; no longer U$7.P$9
- net QEI3_A: now also J53.P$1, U$1.P$6; no longer U$7.P$1
- net QEI3_B: now also J54.P$1, U$1.P$5; no longer U$7.P$3
- net QEI3_Z: now also J55.P$1, U$1.P$4; no longer U$7.P$4
- net RX0: now also J60.P$1
- net RX1: now also J62.P$1, U$11.P$9; no longer U$2.P$5
- net RX2: now also J64.P$1, U$2.P$5; no longer U$2.P$7
- net RX3°: now also CON15.2, U$11.P$14; no longer UART3.2
- net S0: now also J26.P$1
- net S1: now also J27.P$1
- net S2: now also J35.P$1
- net S3: now also J36.P$1
- net S4: now also J37.P$1
- net S5: now also J38.P$1
- net S6: now also J39.P$1
- net S7: now also J40.P$1
- net SCL0: now also J77.P$1, R12.1, U$4.P$4; no longer R2.1, U$5.P$3
- net SCL1: now also J80.P$1, R15.1, U$1.P$9; no longer R4.1, U$5.P$6
- net SCLK0: now also J70.P$1, U$2.P$9; no longer U$4.P$4
- net SCLK1: now also J74.P$1, U$11.P$5; no longer U$4.P$8
- net SDA0: now also J76.P$1, R11.1, U$4.P$1; no longer R1.1, U$5.P$1
- net SDA1: now also J79.P$1, R16.1, U$1.P$7; no longer R3.1, U$5.P$5
- net TX0: now also J59.P$1
- net TX1: now also J61.P$1, U$11.P$8; no longer U$2.P$4
- net TX2: now also J63.P$1, U$2.P$4; no longer U$2.P$6
- net TX3°: now also CON15.3, U$11.P$15; no longer UART3.3
- net WIFI0_WPS: now also J96.P$1
- net WIFI1_WPS: now also J117.P$1
Routing:
- net A12V: track 0.00 -> 303.6 mm, vias 0 -> 18
- net A5V: track 0.00 -> 179.5 mm, vias 0 -> 3
- net 24V: track 0.00 -> 163.8 mm, vias 0 -> 21
- net 5V: track 0.00 -> 121.6 mm, vias 0 -> 6
- net GND: track 37.5 -> 157.1 mm, vias 0 -> 272
- net AD0_VREF: track 0.00 -> 86.0 mm, vias 0 -> 5
- net N$63: track 0.00 -> 83.1 mm, vias 0 -> 1
- net ESC_PWR: track 0.00 -> 38.7 mm, vias 0 -> 2
- net N$196: track 0.00 -> 32.8 mm, vias 0 -> 1
- net ESC0_PWM°: track 0.00 -> 30.1 mm, vias 0 -> 2
- net N$52: track 0.00 -> 29.9 mm, vias 0 -> 1
- net N$182: track 0.00 -> 28.0 mm
- net N$206: track 27.5 -> 0.00 mm
- net N$6: track 0.00 -> 26.7 mm, vias 0 -> 2
- net N$193: track 0.00 -> 23.7 mm
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- added copper zone on layer 1, net GND
- added copper zone on layer 15, net GND
- added copper zone on layer 16, net GND
- added copper zone on layer 2, net GND
Other:
- board size 152 x 190.6 mm -> 210 x 130 mm
