File: hardware/expansion_board_V0/expansion_board_V0.brd (EAGLE design)
At the start: 210 x 130 mm, 550 parts, among them CON1 M2, CON10 QEI3, CON11 QEI2, CON12 CON14, CON13 UART1, CON14 UART0, CON15 BALISE, CON2 TELEM, CON28 NC, CON3 M5, CON4 M3, CON5 M4, CON6 M0, CON7 M1, CON8 QEI1, CON9 QEI0, IC1 REF5025I, IC2 REF5030I, J1 0, J10 0, J100 JUMP_402, J101 JUMP_402, J102 JUMP_402, J103 JUMP_402, J104 JUMP_402, J105 JUMP_402, J106 JUMP_402, J107 JUMP_402, J108 JUMP_402, J109 JUMP_402, J11 0, J110 JUMP_402, J111 JUMP_402, J112 JUMP_402, J113 JUMP_402, J114 JUMP_402, J115 JUMP_402, J116 JUMP_402, J117 JUMP_402, J118 JUMP_402, J119 nc, J12 0, J120 0, J121 nc, J122 0, J123 nc, J124 0, J125 nc, J126 0, J127 nc, J128 0, J129 nc, J13 0, J130 0, J131 nc, J132 0, J14 0, J15 0, J16 0, J17 0, J19 0, J2 0, J20 nc, J21 0, J22 0, J23 0, J24 nc, J25 nc, J26 JUMP_402, J27 JUMP_402, J28 nc, J29 0, J3 0, J30 0, J31 nc, J32 0, J33 0, J34 0, J35 JUMP_402, J36 JUMP_402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

Commit message: Add Gemicom lib + update module in sch/brd
Parts:
- removed U$12, U$35: LGA22U, Gemicom:LGA22U
- added U$5, U$6: LGA22U, Gemicom:LGA22U
Connections:
- net 3V3: now also U$5.P$6, U$6.P$6; no longer U$12.P$6, U$35.P$6
- net GND: now also U$5.P$1, U$5.P$10, U$5.P$11, U$5.P$12, U$5.P$13, U$5.P$14, U$5.P$15, U$5.P$16, U$5.P$17, U$5.P$18, U$5.P$7, U$5.P$8, U$5.P$9, U$6.P$1, U$6.P$10, U$6.P$11, U$6.P$12, U$6.P$13, U$6.P$14, U$6.P$15, U$6.P$16, U$6.P$17, U$6.P$18, U$6.P$7, U$6.P$8, U$6.P$9; no longer U$12.P$1, U$12.P$10, U$12.P$11, U$12.P$12, U$12.P$13, U$12.P$14, U$12.P$15, U$12.P$16, U$12.P$17, U$12.P$18, U$12.P$7, U$12.P$8, U$12.P$9, U$35.P$1, U$35.P$10, U$35.P$11, U$35.P$12, U$35.P$13, U$35.P$14, U$35.P$15, U$35.P$16, U$35.P$17, U$35.P$18, U$35.P$7, U$35.P$8, U$35.P$9
- net WIFI0_DM: now also U$5.P$5; no longer U$12.P$5
- net WIFI0_DP: now also U$5.P$4; no longer U$12.P$4
- net WIFI0_LED: now also U$5.P$3; no longer U$12.P$3
- net WIFI0_WPS: now also U$5.P$2; no longer U$12.P$2
- net WIFI1_DM: now also U$6.P$5; no longer U$35.P$5
- net WIFI1_DP: now also U$6.P$4; no longer U$35.P$4
- net WIFI1_LED: now also U$6.P$3; no longer U$35.P$3
- net WIFI1_WPS: now also U$6.P$2; no longer U$35.P$2

Commit message: -
Parts:
- added CON16, CON17: CON10_2_2.54, iocene:CON245P2030X890-2X5N
- added J133: NC, iocene:JUMC1608X50AN
- moved U$5 335.8 mm to (-25.2, 58.0), turned to 270 degrees
- moved U$6 313.4 mm to (-25.3, -35.1), turned to 270 degrees
- moved T3 158.9 mm to (-113.2, 49.5)
- moved D2 148.8 mm to (-28.3, -69.9)
- moved D6 148.7 mm to (-28.3, -72.7)
- moved D5 147.5 mm to (-29.4, -74.9)
- moved D7 147.4 mm to (-29.7, -78.7)
- moved R99 147.2 mm to (-70.5, -85.8)
- moved C183 147.2 mm to (-71.5, -83.8)
- moved C30 147.2 mm to (-73.7, -82.5)
- moved C31 147.2 mm to (-76.0, -85.1)
- moved R100 147.2 mm to (-71.5, -85.9)
- moved U17 147.2 mm to (-73.5, -85.2)
- moved R108 146.1 mm to (-34.0, -72.3)
- moved R107 145.6 mm to (-34.9, -69.2)
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Connections:
- net 12V: now also J133.P$2
- net 5V: now also CON16.P$9, CON17.P$9
- net A12V: now also J133.P$1
- net A5V: now also CON16.P$2, CON17.P$2
- net AD0_VREF: now also CON16.P$10, CON17.P$10
- net ESC0_CS: now also CON16.P$7, CON17.P$7
- net ESC0_DIR°: now also CON16.P$3, CON17.P$3
- net ESC0_PWM°: now also CON16.P$5, CON17.P$5
- net ESC1_CS: now also CON16.P$8, CON17.P$8
- net ESC1_DIR°: now also CON16.P$4, CON17.P$4
- net ESC1_PWM°: now also CON16.P$1, CON17.P$1
- net GND: now also CON16.P$6, CON17.P$6
Routing:
- net A12V: track 303.6 -> 313.9 mm
- net A5V: track 179.5 -> 170.3 mm, vias 3 -> 2
- net S0°: track 0.00 -> 7.92 mm
- net S1°: track 0.00 -> 5.32 mm
- net S2°: track 0.00 -> 2.71 mm
- net N$45: track 16.2 -> 17.3 mm
- net N$44: track 17.9 -> 19.0 mm
- net N$23: track 23.4 -> 24.5 mm
- net N$21: track 23.5 -> 24.6 mm
- net N$6: track 26.7 -> 27.7 mm
- net N$43: track 19.8 -> 20.8 mm
- net N$47: track 14.4 -> 15.4 mm
- net ESC1_CS: track 6.70 -> 6.62 mm, vias 2 -> 1
- net 5V: vias 6 -> 5
- net ESC0_PWM°: track 30.1 -> 30.2 mm, vias 2 -> 1
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
Commit message: Update connector placement fo match Nano SOC board
Parts:
- moved J18 1.80 mm to (-13.7, -30.4)
- moved JP7_GPIO1 1.80 mm to (-59.4, -30.6)
- moved CON17 0.50 mm to (-86.1, -4.60)
- moved U4 0.50 mm to (-101.1, -26.1)
- moved UW1 0.50 mm to (-91.1, -2.17)
- moved UW2 0.50 mm to (-89.0, 4.12)

Commit message: -
Parts:
- removed C159: 100n, iocene:CAPC1005X55N
- removed C171: 10n, iocene:CAPC1005X55N
- removed D2: LED_603, iocene:LEDC1608X60N
- removed R107: 330, iocene:RESC1005X40N
- added D8, D9: LED_603, iocene:LEDC1608X60N
- added J134, J135: JUMP_402, iocene:JUMC1005X50N
- added R1, R2: 560, iocene:RESC1005X40N
- moved J93 330.0 mm to (-59.4, 24.5), flipped to the bottom, turned to 270 degrees
- moved J94 329.1 mm to (-83.8, -33.2), turned to 90 degrees
- moved J95 329.0 mm to (-83.6, -30.3), turned to 90 degrees
- moved J82 324.8 mm to (-78.2, 33.0), turned to 270 degrees
- moved J116 323.4 mm to (-55.2, 23.9), flipped to the bottom, turned to 270 degrees
- moved J113 323.1 mm to (-53.1, 24.1), flipped to the bottom, turned to 270 degrees
- moved J84 322.1 mm to (-83.6, 32.9), turned to 270 degrees
- moved J85 320.7 mm to (-75.8, 33.1), turned to 270 degrees
- moved J115 320.4 mm to (-49.9, 23.9), flipped to the bottom, turned to 270 degrees
- moved J86 318.7 mm to (-81.0, 32.9), turned to 270 degrees
- moved J83 314.3 mm to (-73.6, 33.0), turned to 270 degrees
- moved J114 312.6 mm to (-47.4, 23.8), flipped to the bottom, turned to 270 degrees
- moved J65 273.7 mm to (-62.3, 24.3), flipped to the bottom, turned to 270 degrees
- moved J118 254.9 mm to (-45.0, 24.1), flipped to the bottom, turned to 270 degrees
- moved C166 211.3 mm to (-97.0, 27.1), turned to 90 degrees
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Connections:
- removed net N$203: D2.A, R107.2
- new net AD0_VREF*: C174.2, C180.2, CON16.P$10, U$31.P$6, U$31.P$7, U$34.P$6, U$34.P$7
- new net ESC0_CS*: CON16.P$7, R93.2
- new net ESC0_DIR°*: CON16.P$3, T1.P$1
- new net ESC0_PWM°*: CON16.P$5, U14.PWM
- new net ESC1_CS*: CON16.P$8, R95.2
- new net ESC1_DIR°*: CON16.P$4, T2.P$1
- new net ESC1_PWM°*: CON16.P$1, U16.PWM
- new net LEDA: J134.P$1, R2.1
- new net LEDB: J135.P$1, R1.1
- new net N$61: D8.A, R1.2
- new net N$64: D9.A, R2.2
- net 12V: now also R112.1; no longer J31.P$1, R116.1
- net 24V: now also R116.1; no longer R114.1
- net 3V3: no longer R107.1
- net 5V: no longer C210.1, U20.16
- net A12V: now also J31.P$1
- net A5V: now also R114.1; no longer R112.1
- net AD0_VREF: no longer C171.2, C174.2, C180.2, CON16.P$10, U$31.P$6, U$31.P$7, U$34.P$6, U$34.P$7, UV1.4
- net BALISE: now also U$10.P$9
- net BALISE°: now also U$10.P$12
- net BUZZER: now also U$10.P$3; no longer U$10.P$6
- net BUZZER°: now also U$10.P$18; no longer U$10.P$15
- net D3V3: now also C210.1, U20.16; no longer C159.2
- net ESC0_CS: now also C179.2, UV1.63; no longer C173.2, CON16.P$7, R93.2, UV1.49
- net ESC0_DIR: now also U$10.P$6; no longer U$10.P$3
- net ESC0_DIR°: now also U$10.P$15; no longer CON16.P$3, T1.P$1, U$10.P$18
- net ESC0_PWM: now also U$10.P$7; no longer U$10.P$1
- net ESC0_PWM°: now also U$10.P$14; no longer CON16.P$5, U$10.P$20, U14.PWM
- net ESC1_CS: now also C173.2, UV1.1; no longer C179.2, CON16.P$8, R95.2, UV1.47
- net ESC1_DIR: now also U$10.P$5; no longer U$10.P$9
- net ESC1_DIR°: now also U$10.P$16; no longer CON16.P$4, T2.P$1, U$10.P$12
- net ESC1_PWM: now also U$10.P$4; no longer U$10.P$8
- net ESC1_PWM°: now also U$10.P$17; no longer CON16.P$1, U$10.P$13, U16.PWM
- net GND: now also D8.C, D9.C, UV1.4; no longer C159.1, C171.1, D2.C
- net LOW_VOLTAGE: now also UV1.3; no longer UV1.45
- net M0_CS: now also UV1.47; no longer UV1.3
- net M1_CS: now also UV1.45; no longer UV1.1
- net M2_CS: now also UV1.49; no longer UV1.63
- net M3_CS: now also UV1.51; no longer UV1.61
- net M4_CS: now also UV1.61; no longer UV1.51
- net TELEM: now also U$10.P$1
- net TELEM°: now also U$10.P$20
Routing:
- net 5V: track 121.6 -> 625.8 mm, vias 5 -> 18
- net D3V3: track 0.00 -> 184.7 mm, vias 0 -> 8
- net A5V: track 170.3 -> 328.9 mm, vias 2 -> 4
- net 12V: track 0.00 -> 145.3 mm
- net 24V: track 163.8 -> 263.8 mm, vias 21 -> 25
- net AD0_VREF: track 86.1 -> 186.0 mm, vias 4 -> 8
- net M4_CS: track 10.4 -> 75.5 mm, vias 1 -> 2
- net LOW_VOLTAGE: track 0.00 -> 63.7 mm, vias 0 -> 2
- net A12V: track 313.9 -> 373.0 mm, vias 18 -> 19
- net BUZZER°: track 0.00 -> 47.9 mm, vias 0 -> 1
- net M0_PWMA: track 4.60 -> 45.0 mm
- net M0_FAULT: track 6.35 -> 46.4 mm
- net M3_CS: track 11.1 -> 51.0 mm, vias 1 -> 2
- net M0_PWMB: track 5.76 -> 43.8 mm
- net QEI1_B°: track 0.00 -> 37.8 mm
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
Commit message: -
Parts:
- moved R12 37.9 mm to (-58.1, 28.2), flipped to the top, turned to 270 degrees
- moved R11 36.5 mm to (-55.7, 28.0), flipped to the top, turned to 270 degrees
- moved C12 13.9 mm to (-60.9, 48.6)
- moved J100 12.9 mm to (-45.5, 32.9)
- moved J97 12.8 mm to (-53.1, 30.3)
- moved J109 12.4 mm to (-55.8, 32.7)
- moved J52 10.5 mm to (-65.6, 32.9)
- moved J110 10.3 mm to (-50.6, 30.4)
- moved J51 10.2 mm to (-68.2, 32.8)
- moved J76 10.2 mm to (-55.6, 30.1)
- moved J99 10.1 mm to (-50.4, 32.9)
- moved J98 10.0 mm to (-53.1, 32.9)
- moved C11 8.83 mm to (-95.5, 54.3), turned to 270 degrees
- moved J57 7.81 mm to (-60.7, 30.4)
- moved J77 7.80 mm to (-58.0, 30.1)
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Routing:
- net D3V3: track 184.7 -> 304.3 mm
- net 5V: track 625.8 -> 739.5 mm
- net QEI0_A°: track 0.00 -> 33.2 mm
- net QEI0_B°: track 0.00 -> 30.5 mm
- net SCLK0°: track 0.00 -> 28.6 mm
- net M1_FAULT: track 30.1 -> 57.2 mm
- net M0_PWMB: track 43.8 -> 70.8 mm
- net M1_PWMA: track 28.4 -> 55.4 mm
- net M0_PWMA: track 45.0 -> 72.0 mm
- net M0_FAULT: track 46.4 -> 73.5 mm
- net M1_PWMB: track 27.5 -> 54.5 mm
- net SS0°: track 0.00 -> 26.6 mm
- net BUZZER°: track 47.9 -> 73.6 mm, vias 1 -> 2
- net MOSI0°: track 0.00 -> 24.7 mm
- net M23_FAULT: track 18.8 -> 42.6 mm
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
Commit message: Update WPS and LED on WiFi module
Parts:
- removed J117, J96: JUMP_402, iocene:JUMC1005X50N
- added D10, D11: LED_603, iocene:LEDC1608X60N
- added R3, R7: 10k, iocene:RESC1005X40N
- added R4, R8: 330, iocene:RESC1005X40N
Connections:
- removed net WIFI0_LED: U$5.P$3
- removed net WIFI0_WPS: J96.P$1, U$5.P$2
- new net N$66: D10.C, R4.2
- new net N$67: D11.C, R8.2
- new net WIFI1_LED1: R8.1, U$5.P$3
- new net WIFI1_WPS1: R7.1, U$5.P$2
- net 3V3: now also D10.A, D11.A, R3.2, R7.2
- net WIFI1_LED: now also R4.1
- net WIFI1_WPS: now also R3.1; no longer J117.P$1
Other:
- board text added: "On inverse pas M1 et M0 ?"

Commit message: -
Parts:
- removed J100, J101, J102, J103, J104, J105, J106, J107, J108, J109, J110, J111, J112, J113, J114, J115, J116, J118, J134, J135, J26, J27, J35, J36, J37, J38, J39, J40, J41, J42, J43, J44, J45, J46, J47, J48, J49, J50, J51, J52, J53, J54, J55, J56, J57, J58, J59, J60, J61, J62, J63, J64, J65, J66, J67, J68, J69, J70, J71, J72, J73, J74, J75, J76, J77, J78, J79, J80, J81, J82, J83, J84, J85, J86, J87, J88, J89, J90, J91, J92, J93, J94, J95, J97, J98, J99: JUMP_402, iocene:JUMC1005X50N
- moved D11 301.3 mm to (28.1, 53.2)
- moved R7 297.7 mm to (20.7, 53.4)
- moved R8 292.2 mm to (19.5, 49.1)
- moved D10 258.8 mm to (32.5, -35.5)
- moved R4 252.8 mm to (26.6, -32.7)
- moved R3 250.6 mm to (26.8, -36.6)
- moved C156 1.98 mm to (-37.3, -44.8)
- moved C183 1.98 mm to (-42.0, -42.6)
- moved C30 1.98 mm to (-43.9, -46.5)
- moved C31 1.98 mm to (-37.5, -45.5)
- moved R100 1.98 mm to (-39.4, -42.6)
- moved R99 1.98 mm to (-40.7, -42.6)
- moved U17 1.98 mm to (-40.7, -45.5)
- moved C141 0.50 mm to (-129.7, 37.8)
- moved C161 0.40 mm to (-98.8, 21.3)
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Connections:
- removed net 3V: U4.3V
- removed net ARDUINO_IO0: U4.D0
- removed net ARDUINO_IO1: U4.D1
- removed net ARDUINO_IO10: U4.D10
- removed net ARDUINO_IO11: U4.D11
- removed net ARDUINO_IO12: U4.D12
- removed net ARDUINO_IO13: U4.D13
- removed net ARDUINO_IO2: U4.D2
- removed net ARDUINO_IO3: U4.D3
- removed net ARDUINO_IO4: U4.D4
- removed net ARDUINO_IO5: U4.D5
- removed net ARDUINO_IO6: U4.D6
- removed net ARDUINO_IO7: U4.D7
- removed net ARDUINO_IO8: U4.D8
- removed net ARDUINO_IO9: U4.D9
- removed net GPIO0_0: JP1_GPIO0.1
- removed net GPIO0_1: JP1_GPIO0.2
- removed net GPIO0_10: JP1_GPIO0.13
- removed net GPIO0_11: JP1_GPIO0.14
- removed net GPIO0_12: JP1_GPIO0.15
- removed net GPIO0_13: JP1_GPIO0.16
- removed net GPIO0_14: JP1_GPIO0.17
- removed net GPIO0_15: JP1_GPIO0.18
- removed net GPIO0_16: JP1_GPIO0.19
- removed net GPIO0_17: JP1_GPIO0.20
- removed net GPIO0_18: JP1_GPIO0.21
- removed net GPIO0_19: JP1_GPIO0.22
- removed net GPIO0_2: JP1_GPIO0.3
- removed net GPIO0_20: JP1_GPIO0.23
- removed net GPIO0_21: JP1_GPIO0.24
- removed net GPIO0_22: JP1_GPIO0.25
- removed net GPIO0_23: JP1_GPIO0.26
- removed net GPIO0_24: JP1_GPIO0.27
- removed net GPIO0_25: JP1_GPIO0.28
- removed net GPIO0_26: JP1_GPIO0.31
- removed net GPIO0_27: JP1_GPIO0.32
- removed net GPIO0_28: JP1_GPIO0.33
- removed net GPIO0_29: JP1_GPIO0.34
- removed net GPIO0_3: JP1_GPIO0.4
- removed net GPIO0_30: JP1_GPIO0.35
- removed net GPIO0_31: JP1_GPIO0.36
- removed net GPIO0_32: JP1_GPIO0.37
- removed net GPIO0_33: JP1_GPIO0.38
- removed net GPIO0_34: JP1_GPIO0.39
- removed net GPIO0_35: JP1_GPIO0.40
- removed net GPIO0_4: JP1_GPIO0.5
- removed net GPIO0_5: JP1_GPIO0.6
- removed net GPIO0_6: JP1_GPIO0.7
- removed net GPIO0_7: JP1_GPIO0.8
- removed net GPIO0_8: JP1_GPIO0.9
- removed net GPIO0_9: JP1_GPIO0.10
- removed net GPIO1_0: JP7_GPIO1.1
- removed net GPIO1_1: JP7_GPIO1.2
- removed net GPIO1_10: JP7_GPIO1.13
- removed net GPIO1_11: JP7_GPIO1.14
- removed net GPIO1_12: JP7_GPIO1.15
- removed net GPIO1_13: JP7_GPIO1.16
- removed net GPIO1_14: JP7_GPIO1.17
- removed net GPIO1_15: JP7_GPIO1.18
- removed net GPIO1_16: JP7_GPIO1.19
- removed net GPIO1_17: JP7_GPIO1.20
- removed net GPIO1_18: JP7_GPIO1.21
- removed net GPIO1_19: JP7_GPIO1.22
- removed net GPIO1_2: JP7_GPIO1.3
- removed net GPIO1_20: JP7_GPIO1.23
- removed net GPIO1_21: JP7_GPIO1.24
- removed net GPIO1_22: JP7_GPIO1.25
- removed net GPIO1_23: JP7_GPIO1.26
- removed net GPIO1_24: JP7_GPIO1.27
- removed net GPIO1_25: JP7_GPIO1.28
- removed net GPIO1_26: JP7_GPIO1.31
- removed net GPIO1_27: JP7_GPIO1.32
- removed net GPIO1_28: JP7_GPIO1.33
- removed net GPIO1_29: JP7_GPIO1.34
- removed net GPIO1_3: JP7_GPIO1.4
- removed net GPIO1_30: JP7_GPIO1.35
- removed net GPIO1_31: JP7_GPIO1.36
- removed net GPIO1_32: JP7_GPIO1.37
- removed net GPIO1_33: JP7_GPIO1.38
- removed net GPIO1_34: JP7_GPIO1.39
- removed net GPIO1_35: JP7_GPIO1.40
- removed net GPIO1_4: JP7_GPIO1.5
- removed net GPIO1_5: JP7_GPIO1.6
- removed net GPIO1_6: JP7_GPIO1.7
- removed net GPIO1_7: JP7_GPIO1.8
- removed net GPIO1_8: JP7_GPIO1.9
- removed net GPIO1_9: JP7_GPIO1.10
- removed net VIN: U4.VIN
- new net ARDUINO_A5: U4.A5
- net 5V: no longer U4.5V
- net AD0_CLK: now also JP1_GPIO0.6; no longer J82.P$1
- net AD0_DRDY: now also JP1_GPIO0.10; no longer J83.P$1
- net AD0_MISO: now also JP1_GPIO0.2; no longer J86.P$1
- net AD0_SCLK: now also JP1_GPIO0.8; no longer J85.P$1
- net AD0_SYNC: now also JP1_GPIO0.4; no longer J84.P$1
- net AD1_DRDY: now also U4.D11; no longer J88.P$1
- net AD1_MISO: now also U4.D12; no longer J92.P$1
- net AD1_MOSI: now also U4.D13; no longer J91.P$1
- net AD1_RST: now also U4.SCL; no longer J87.P$1
- net AD1_SCLK: now also U4.SDA; no longer J90.P$1
- net AD1_SS: now also U4.D10; no longer J89.P$1
- net BALISE: now also U4.D3; no longer J118.P$1
- net BUZZER: now also U4.D8; no longer J93.P$1
- net ESC0_DIR: now also U4.D5; no longer J115.P$1
- net ESC0_PWM: now also U4.D4; no longer J114.P$1
- net ESC1_DIR: now also U4.D6; no longer J113.P$1
- net ESC1_PWM: now also U4.D7; no longer J116.P$1
- net I2C0: now also JP1_GPIO0.22; no longer J78.P$1
- net I2C1: now also JP7_GPIO1.24; no longer J81.P$1
- net IO0: now also JP1_GPIO0.17; no longer J41.P$1
- net IO1: now also JP1_GPIO0.15; no longer J42.P$1
- net IO2: now also JP1_GPIO0.13; no longer J43.P$1
- net IO3: now also JP1_GPIO0.9; no longer J44.P$1
- net IO4: now also JP1_GPIO0.7; no longer J45.P$1
- net IO5: now also JP1_GPIO0.5; no longer J46.P$1
- net IO6: now also JP1_GPIO0.3; no longer J47.P$1
- net IO7: now also JP1_GPIO0.1; no longer J48.P$1
- net LEDA: now also JP7_GPIO1.1; no longer J134.P$1
- net LEDB: now also JP7_GPIO1.2; no longer J135.P$1
- net LV_MUXA: now also JP7_GPIO1.40; no longer J94.P$1
- net LV_MUXB: now also JP7_GPIO1.39; no longer J95.P$1
- net M0_FAULT: now also JP1_GPIO0.24; no longer J109.P$1
- net M0_PWMA: now also JP1_GPIO0.25; no longer J97.P$1
- net M0_PWMB: now also JP1_GPIO0.26; no longer J98.P$1
- net M1_FAULT: now also JP1_GPIO0.27; no longer J110.P$1
- net M1_PWMA: now also JP1_GPIO0.28; no longer J99.P$1
- net M1_PWMB: now also JP1_GPIO0.32; no longer J100.P$1
- net M23_FAULT: now also JP7_GPIO1.25; no longer J111.P$1
- net M2_PWMA: now also JP7_GPIO1.19; no longer J101.P$1
- net M2_PWMB: now also JP7_GPIO1.17; no longer J102.P$1
- net M3_PWMA: now also JP7_GPIO1.23; no longer J103.P$1
- net M3_PWMB: now also JP7_GPIO1.21; no longer J104.P$1
- net M45_FAULT: now also JP7_GPIO1.37; no longer J112.P$1
- net M4_PWMA: now also JP7_GPIO1.31; no longer J105.P$1
- net M4_PWMB: now also JP7_GPIO1.27; no longer J106.P$1
- net M5_PWMA: now also JP7_GPIO1.35; no longer J107.P$1
- net M5_PWMB: now also JP7_GPIO1.33; no longer J108.P$1
- net MISO0: now also JP1_GPIO0.36; no longer J68.P$1
- net MISO1: now also JP7_GPIO1.20; no longer J72.P$1
- net MOSI0: now also JP1_GPIO0.35; no longer J69.P$1
- net MOSI1: now also JP7_GPIO1.18; no longer J73.P$1
- net QEI0_A: now also JP1_GPIO0.14; no longer J51.P$1
- net QEI0_B: now also JP1_GPIO0.16; no longer J52.P$1
- net QEI1_A: now also JP7_GPIO1.36; no longer J49.P$1
- net QEI1_B: now also JP7_GPIO1.38; no longer J50.P$1
- net QEI2_A: now also JP1_GPIO0.18; no longer J56.P$1
- net QEI2_B: now also JP1_GPIO0.19; no longer J57.P$1
- net QEI2_Z: now also JP1_GPIO0.20; no longer J58.P$1
- net QEI3_A: now also JP7_GPIO1.28; no longer J53.P$1
- net QEI3_B: now also JP7_GPIO1.32; no longer J54.P$1
- net QEI3_Z: now also JP7_GPIO1.34; no longer J55.P$1
- net RX0: now also JP1_GPIO0.39; no longer J60.P$1
- net RX1: now also JP7_GPIO1.4; no longer J62.P$1
- net RX2: now also JP1_GPIO0.37; no longer J64.P$1
- net RX3: now also JP7_GPIO1.8; no longer J67.P$1
- net S0: now also JP7_GPIO1.15; no longer J26.P$1
- net S1: now also JP7_GPIO1.13; no longer J27.P$1
- net S2: now also JP7_GPIO1.9; no longer J35.P$1
- net S3: now also JP7_GPIO1.7; no longer J36.P$1
- net S4: now also JP7_GPIO1.5; no longer J37.P$1
- net S5: now also U4.D0; no longer J38.P$1
- net S6: now also U4.D1; no longer J39.P$1
- net S7: now also U4.D2; no longer J40.P$1
- net SCL0: now also JP1_GPIO0.21; no longer J77.P$1
- net SCL1: now also JP7_GPIO1.22; no longer J80.P$1
- net SCLK0: now also JP1_GPIO0.33; no longer J70.P$1
- net SCLK1: now also JP7_GPIO1.14; no longer J74.P$1
- net SDA0: now also JP1_GPIO0.23; no longer J76.P$1
- net SDA1: now also JP7_GPIO1.26; no longer J79.P$1
- net SS0: now also JP1_GPIO0.34; no longer J71.P$1
- net SS1: now also JP7_GPIO1.16; no longer J75.P$1
- net TELEM: now also U4.D9; no longer J65.P$1
- net TX0: now also JP1_GPIO0.40; no longer J59.P$1
- net TX1: now also JP7_GPIO1.6; no longer J61.P$1
- net TX2: now also JP1_GPIO0.38; no longer J63.P$1
- net TX3: now also JP7_GPIO1.10; no longer J66.P$1
Routing:
- net TELEM°: track 0.00 -> 76.0 mm, vias 0 -> 1
- net BALISE°: track 0.00 -> 65.6 mm, vias 0 -> 1
- net S5: track 0.00 -> 61.2 mm
- net S6: track 0.00 -> 59.0 mm
- net S7: track 0.00 -> 57.0 mm
- net D3V3: track 304.3 -> 358.4 mm, vias 8 -> 9
- net SDA0: track 0.00 -> 47.4 mm
- net S4: track 0.00 -> 47.0 mm
- net BALISE: track 0.00 -> 44.3 mm
- net S3: track 0.00 -> 44.2 mm
- net SCL0: track 0.00 -> 44.0 mm
- net S2: track 0.00 -> 41.4 mm
- net ESC0_PWM: track 0.00 -> 41.2 mm
- net I2C0: track 0.00 -> 40.5 mm
- net QEI2_B: track 0.00 -> 39.2 mm
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