File: hardware/expansion_board_V0/expansion_board_V0.sch (EAGLE design)
At the start: 559 parts, among them CON1 M2, CON10 QEI3, CON11 QEI2, CON12 CON14, CON13 UART1, CON14 UART0, CON15 BALISE, CON16 CON10_2_2.54, CON17 CON10_2_2.54, CON2 TELEM, CON28 NC, CON3 M5, CON4 M3, CON5 M4, CON6 M0, CON7 M1, CON8 QEI1, CON9 QEI0, IC1 REF5025I, IC2 REF5030I, J1 0, J10 0, J100 JUMP_402, J101 JUMP_402, J102 JUMP_402, J103 JUMP_402, J104 JUMP_402, J105 JUMP_402, J106 JUMP_402, J107 JUMP_402, J108 JUMP_402, J109 JUMP_402, J11 0, J110 JUMP_402, J111 JUMP_402, J112 JUMP_402, J113 JUMP_402, J114 JUMP_402, J115 JUMP_402, J116 JUMP_402, J118 JUMP_402, J119 nc, J12 0, J120 0, J121 nc, J122 0, J123 nc, J124 0, J125 nc, J126 0, J127 nc, J128 0, J129 nc, J13 0, J130 0, J131 nc, J132 0, J133 NC, J134 JUMP_402, J135 JUMP_402, J14 0, J15 0, J16 0, J17 0, J19 0, J2 0, J20 nc, J21 0, J22 0, J23 0, J24 nc, J25 nc, J26 JUMP_402, J27 JUMP_402, J28 nc, J29 0, J3 0, J30 0, J31 nc, J32 0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

Commit message: -
Parts:
- removed J100, J101, J102, J103, J104, J105, J106, J107, J108, J109, J110, J111, J112, J113, J114, J115, J116, J118, J134, J135, J26, J27, J35, J36, J37, J38, J39, J40, J41, J42, J43, J44, J45, J46, J47, J48, J49, J50, J51, J52, J53, J54, J55, J56, J57, J58, J59, J60, J61, J62, J63, J64, J65, J66, J67, J68, J69, J70, J71, J72, J73, J74, J75, J76, J77, J78, J79, J80, J81, J82, J83, J84, J85, J86, J87, J88, J89, J90, J91, J92, J93, J94, J95, J97, J98, J99: JUMP_402, iocene:JUMP_402
Connections:
- removed net ARDUINO_IO0: U4.D0
- removed net ARDUINO_IO1: U4.D1
- removed net ARDUINO_IO10: U4.D10
- removed net ARDUINO_IO11: U4.D11
- removed net ARDUINO_IO12: U4.D12
- removed net ARDUINO_IO13: U4.D13
- removed net ARDUINO_IO2: U4.D2
- removed net ARDUINO_IO3: U4.D3
- removed net ARDUINO_IO4: U4.D4
- removed net ARDUINO_IO5: U4.D5
- removed net ARDUINO_IO6: U4.D6
- removed net ARDUINO_IO7: U4.D7
- removed net ARDUINO_IO8: U4.D8
- removed net ARDUINO_IO9: U4.D9
- removed net GPIO0_0: JP1_GPIO0.1
- removed net GPIO0_1: JP1_GPIO0.2
- removed net GPIO0_10: JP1_GPIO0.13
- removed net GPIO0_11: JP1_GPIO0.14
- removed net GPIO0_12: JP1_GPIO0.15
- removed net GPIO0_13: JP1_GPIO0.16
- removed net GPIO0_14: JP1_GPIO0.17
- removed net GPIO0_15: JP1_GPIO0.18
- removed net GPIO0_16: JP1_GPIO0.19
- removed net GPIO0_17: JP1_GPIO0.20
- removed net GPIO0_18: JP1_GPIO0.21
- removed net GPIO0_19: JP1_GPIO0.22
- removed net GPIO0_2: JP1_GPIO0.3
- removed net GPIO0_20: JP1_GPIO0.23
- removed net GPIO0_21: JP1_GPIO0.24
- removed net GPIO0_22: JP1_GPIO0.25
- removed net GPIO0_23: JP1_GPIO0.26
- removed net GPIO0_24: JP1_GPIO0.27
- removed net GPIO0_25: JP1_GPIO0.28
- removed net GPIO0_26: JP1_GPIO0.31
- removed net GPIO0_27: JP1_GPIO0.32
- removed net GPIO0_28: JP1_GPIO0.33
- removed net GPIO0_29: JP1_GPIO0.34
- removed net GPIO0_3: JP1_GPIO0.4
- removed net GPIO0_30: JP1_GPIO0.35
- removed net GPIO0_31: JP1_GPIO0.36
- removed net GPIO0_32: JP1_GPIO0.37
- removed net GPIO0_33: JP1_GPIO0.38
- removed net GPIO0_34: JP1_GPIO0.39
- removed net GPIO0_35: JP1_GPIO0.40
- removed net GPIO0_4: JP1_GPIO0.5
- removed net GPIO0_5: JP1_GPIO0.6
- removed net GPIO0_6: JP1_GPIO0.7
- removed net GPIO0_7: JP1_GPIO0.8
- removed net GPIO0_8: JP1_GPIO0.9
- removed net GPIO0_9: JP1_GPIO0.10
- removed net GPIO1_0: JP7_GPIO1.1
- removed net GPIO1_1: JP7_GPIO1.2
- removed net GPIO1_10: JP7_GPIO1.13
- removed net GPIO1_11: JP7_GPIO1.14
- removed net GPIO1_12: JP7_GPIO1.15
- removed net GPIO1_13: JP7_GPIO1.16
- removed net GPIO1_14: JP7_GPIO1.17
- removed net GPIO1_15: JP7_GPIO1.18
- removed net GPIO1_16: JP7_GPIO1.19
- removed net GPIO1_17: JP7_GPIO1.20
- removed net GPIO1_18: JP7_GPIO1.21
- removed net GPIO1_19: JP7_GPIO1.22
- removed net GPIO1_2: JP7_GPIO1.3
- removed net GPIO1_20: JP7_GPIO1.23
- removed net GPIO1_21: JP7_GPIO1.24
- removed net GPIO1_22: JP7_GPIO1.25
- removed net GPIO1_23: JP7_GPIO1.26
- removed net GPIO1_24: JP7_GPIO1.27
- removed net GPIO1_25: JP7_GPIO1.28
- removed net GPIO1_26: JP7_GPIO1.31
- removed net GPIO1_27: JP7_GPIO1.32
- removed net GPIO1_28: JP7_GPIO1.33
- removed net GPIO1_29: JP7_GPIO1.34
- removed net GPIO1_3: JP7_GPIO1.4
- removed net GPIO1_30: JP7_GPIO1.35
- removed net GPIO1_31: JP7_GPIO1.36
- removed net GPIO1_32: JP7_GPIO1.37
- removed net GPIO1_33: JP7_GPIO1.38
- removed net GPIO1_34: JP7_GPIO1.39
- removed net GPIO1_35: JP7_GPIO1.40
- removed net GPIO1_4: JP7_GPIO1.5
- removed net GPIO1_5: JP7_GPIO1.6
- removed net GPIO1_6: JP7_GPIO1.7
- removed net GPIO1_7: JP7_GPIO1.8
- removed net GPIO1_8: JP7_GPIO1.9
- removed net GPIO1_9: JP7_GPIO1.10
- new net ARDUINO_A5: U4.A5/SCL
- net AD0_CLK: now also JP1_GPIO0.6; no longer J82.1
- net AD0_DRDY: now also JP1_GPIO0.10; no longer J83.1
- net AD0_MISO: now also JP1_GPIO0.2; no longer J86.1
- net AD0_SCLK: now also JP1_GPIO0.8; no longer J85.1
- net AD0_SYNC: now also JP1_GPIO0.4; no longer J84.1
- net AD1_DRDY: now also U4.D11; no longer J88.1
- net AD1_MISO: now also U4.D12; no longer J92.1
- net AD1_MOSI: now also U4.D13; no longer J91.1
- net AD1_RST: now also U4.SCL; no longer J87.1
- net AD1_SCLK: now also U4.SDA; no longer J90.1
- net AD1_SS: now also U4.D10; no longer J89.1
- net BALISE: now also U4.D3; no longer J118.1
- net BUZZER: now also U4.D8; no longer J93.1
- net ESC0_DIR: now also U4.D5; no longer J115.1
- net ESC0_PWM: now also U4.D4; no longer J114.1
- net ESC1_DIR: now also U4.D6; no longer J113.1
- net ESC1_PWM: now also U4.D7; no longer J116.1
- net I2C0: now also JP1_GPIO0.22; no longer J78.1
- net I2C1: now also JP7_GPIO1.24; no longer J81.1
- net IO0: now also JP1_GPIO0.17; no longer J41.1
- net IO1: now also JP1_GPIO0.15; no longer J42.1
- net IO2: now also JP1_GPIO0.13; no longer J43.1
- net IO3: now also JP1_GPIO0.9; no longer J44.1
- net IO4: now also JP1_GPIO0.7; no longer J45.1
- net IO5: now also JP1_GPIO0.5; no longer J46.1
- net IO6: now also JP1_GPIO0.3; no longer J47.1
- net IO7: now also JP1_GPIO0.1; no longer J48.1
- net LEDA: now also JP7_GPIO1.1; no longer J134.1
- net LEDB: now also JP7_GPIO1.2; no longer J135.1
- net LV_MUXA: now also JP7_GPIO1.40; no longer J94.1
- net LV_MUXB: now also JP7_GPIO1.39; no longer J95.1
- net M0_FAULT: now also JP1_GPIO0.24; no longer J109.1
- net M0_PWMA: now also JP1_GPIO0.25; no longer J97.1
- net M0_PWMB: now also JP1_GPIO0.26; no longer J98.1
- net M1_FAULT: now also JP1_GPIO0.27; no longer J110.1
- net M1_PWMA: now also JP1_GPIO0.28; no longer J99.1
- net M1_PWMB: now also JP1_GPIO0.32; no longer J100.1
- net M23_FAULT: now also JP7_GPIO1.25; no longer J111.1
- net M2_PWMA: now also JP7_GPIO1.19; no longer J101.1
- net M2_PWMB: now also JP7_GPIO1.17; no longer J102.1
- net M3_PWMA: now also JP7_GPIO1.23; no longer J103.1
- net M3_PWMB: now also JP7_GPIO1.21; no longer J104.1
- net M45_FAULT: now also JP7_GPIO1.37; no longer J112.1
- net M4_PWMA: now also JP7_GPIO1.31; no longer J105.1
- net M4_PWMB: now also JP7_GPIO1.27; no longer J106.1
- net M5_PWMA: now also JP7_GPIO1.35; no longer J107.1
- net M5_PWMB: now also JP7_GPIO1.33; no longer J108.1
- net MISO0: now also JP1_GPIO0.36; no longer J68.1
- net MISO1: now also JP7_GPIO1.20; no longer J72.1
- net MOSI0: now also JP1_GPIO0.35; no longer J69.1
- net MOSI1: now also JP7_GPIO1.18; no longer J73.1
- net QEI0_A: now also JP1_GPIO0.14; no longer J51.1
- net QEI0_B: now also JP1_GPIO0.16; no longer J52.1
- net QEI1_A: now also JP7_GPIO1.36; no longer J49.1
- net QEI1_B: now also JP7_GPIO1.38; no longer J50.1
- net QEI2_A: now also JP1_GPIO0.18; no longer J56.1
- net QEI2_B: now also JP1_GPIO0.19; no longer J57.1
- net QEI2_Z: now also JP1_GPIO0.20; no longer J58.1
- net QEI3_A: now also JP7_GPIO1.28; no longer J53.1
- net QEI3_B: now also JP7_GPIO1.32; no longer J54.1
- net QEI3_Z: now also JP7_GPIO1.34; no longer J55.1
- net RX0: now also JP1_GPIO0.39; no longer J60.1
- net RX1: now also JP7_GPIO1.4; no longer J62.1
- net RX2: now also JP1_GPIO0.37; no longer J64.1
- net RX3: now also JP7_GPIO1.8; no longer J67.1
- net S0: now also JP7_GPIO1.15; no longer J26.1
- net S1: now also JP7_GPIO1.13; no longer J27.1
- net S2: now also JP7_GPIO1.9; no longer J35.1
- net S3: now also JP7_GPIO1.7; no longer J36.1
- net S4: now also JP7_GPIO1.5; no longer J37.1
- net S5: now also U4.D0; no longer J38.1
- net S6: now also U4.D1; no longer J39.1
- net S7: now also U4.D2; no longer J40.1
- net SCL0: now also JP1_GPIO0.21; no longer J77.1
- net SCL1: now also JP7_GPIO1.22; no longer J80.1
- net SCLK0: now also JP1_GPIO0.33; no longer J70.1
- net SCLK1: now also JP7_GPIO1.14; no longer J74.1
- net SDA0: now also JP1_GPIO0.23; no longer J76.1
- net SDA1: now also JP7_GPIO1.26; no longer J79.1
- net SS0: now also JP1_GPIO0.34; no longer J71.1
- net SS1: now also JP7_GPIO1.16; no longer J75.1
- net TELEM: now also U4.D9; no longer J65.1
- net TX0: now also JP1_GPIO0.40; no longer J59.1
- net TX1: now also JP7_GPIO1.6; no longer J61.1
- net TX2: now also JP1_GPIO0.38; no longer J63.1
- net TX3: now also JP7_GPIO1.10; no longer J66.1
Other:
- note removed: "Arduino I014"
- note removed: "Arduino I015"

Commit message: -
Parts:
- removed AN2: AN2, iocene:CON3_SMT
- removed C195, C205, C206, C207, C208, C210: 100n, iocene:C_402
- removed C196, C198, C199, C200, C201, C202, C203, C204: 1n, iocene:C_402
- removed C209: 100p, iocene:C_402
- removed D11: LED_603, iocene:LED_603
- removed ESC0: ESC0, iocene:CON4_3.81
- removed ESC1: ESC1, iocene:CON4_3.81
- removed FPGA_POWER: FPGApower, iocene:CON2_3.81
- removed J119: nc, iocene:JUMP_402
- removed J120: 0, iocene:JUMP_402
- removed J133: NC, iocene:JUMP_603
- removed L11, L12: SRN2512-R24M, iocene:INDUCTANCE_2520
- removed L13: 600, iocene:INDUCTANCE_603
- removed L14: NC, iocene:INDUCTANCE_603
- removed LIPO_ELEC, LIPO_MOTEUR, LIPO_MOTEUR1, LIPO_MOTEUR2, LIPO_MOTEUR3, LIPO_SERVO: CON2_3.81, iocene:CON2_3.81
- removed R108: 560, iocene:R_402
- removed R109, R113, R117, R118, R119: 5k, iocene:R_402
- removed R112, R114, R115, R116: 100k, iocene:R_402
- removed U$20, U$24: DRV8432, iocene:DRV84X2_DRV8432
- removed U$22, U$31, U$34: INA240-A2, Texas Instruments_By_element14_Batch_1:INA240-TSSOP
- removed U$5: LGA22U, Gemicom:LGA22U
- removed UV1: ADS1278, IMU:ADS1278"
- removed UW1: ADS1258, IMU:ADS1258
- added C103, C138, C152, C159, C171: 100n, iocene:C_402
- added C151: 18p, iocene:C_402
- added C153: 2.2u, iocene:C_603
- added C175: 1u, iocene:C_603
- added C176, C24: 10u, iocene:C_805
- added C177: 10n, iocene:C_402
- added C26: 470u, iocene:CPOL
- added C81, C82: 1µ, iocene:C_603
- added CON18: UART0, iocene:CON5_2.54S
- added CON19: QEI1, iocene:CON5_2.54S
- added CON26: UART1, iocene:CON5_2.54S
- added CON27: QEI0, iocene:CON5_2.54S
- added CON31: TELEM, iocene:CON5_2.54S
- added CON32: QEI3, iocene:CON5_2.54S
- added CON36: BALISE, iocene:CON5_2.54S
- added CON41: QEI2, iocene:CON5_2.54S
- added CON56: CON3_2.54S, iocene:CON3_2.54S
- added CON59: CON14, iocene:CON14
- added D2: SMP12A, iocene:ZENER
- added IC3: REF5030I, IMU:REF5025I
- added IC4: REF5025I, IMU:REF5025I
- added J26: 0, iocene:JUMP_402
- added J27: nc, iocene:JUMP_402
- added J47: (no value), SparkFun-Connectors:M05X2NO_SILK
- added L1, L5, L6: SRN2512-R24M, iocene:INDUCTANCE_2520
- added R17, R19: 100k, iocene:R_402
- added R18: 19k, iocene:R_402
- added R27, R31, R81, R91: 10k, iocene:R_402
- added R29: ULR15S-R0055FT2, iocene:R_ULR15S-R0055FT2
- added R33: 30k, iocene:R_402
- added R51: 1k, iocene:R_402
- added U1: SN74LV4052A_SO, iocene:SN74LV4052A_SO
- added U23: LP5900_2.2, iocene:REG_EN_LP5900
- added U24: OPA376, iocene:OPA376
- added U29: ARDUINOR3-DIMENSION, adafruit:ARDUINOR3-DIMENSION
- added U5, U6: TPS82130, iocene:TPS82130
- C100, C101, C102, C106, C107, C113, C114, C115, C116, C117, C122, C123, C129, C130, C131, C132, C75, C98, C99: device iocene:C_603 -> iocene:C_402
- C104, C105, C76: value 100n -> 1n; device iocene:C_603 -> iocene:C_402
- C108, C109, C124, C125, C93, C94: value 1µ -> 100n; device iocene:C_603 -> iocene:C_402
- C11: device iocene:C_402 -> iocene:C_805
- C110, C111, C126, C127, C95, C96: value 1µ -> 1n; device iocene:C_603 -> iocene:C_402
- C118, C133, C136, C173, C192: value 1n -> 100n
- C12: value 100n -> 220u; device iocene:C_402 -> iocene:CPOL
- C121: value 10n -> 1n
- C128, C56, C58, C90: value 100n -> 1n
- C13, C14, C16, C17, C20, C21, C25: value 100n -> 10u; device iocene:C_402 -> iocene:C_805
- C135, C174, C193: value 10n -> 100n
- C141: value 220u -> 100n; device iocene:CPOL -> iocene:C_402
- C148, C158: value 100n -> 2.2u; device iocene:C_402 -> iocene:C_603
- C15, C2, C22, C6: value 100n -> 470u; device iocene:C_402 -> iocene:CPOL
- C150: value 100n -> 18p
- C156, C181, C186, C190, C89: value 470u -> 100n; device iocene:CPOL -> iocene:C_402
- C168: value 10u -> 22n; device iocene:C_805 -> iocene:C_402
- C169: value 1u -> 22n; device iocene:C_603 -> iocene:C_402
- C170: value 100n -> 22n
- C178, C4: value 100n -> 100p
- C179: value 1n -> 1u; device iocene:C_402 -> iocene:C_603
- C18: value 2.2u -> 470u; device iocene:C_603 -> iocene:CPOL
- C180: value 10n -> 10u; device iocene:C_402 -> iocene:C_805
- C182, C184, C185, C188, C189, C28: value 10u -> 100n; device iocene:C_805 -> iocene:C_402
- C183, C187, C191: value nc -> 100n
- C19, C23, C27: value 100n -> nc
- C29, C32, C38, C41: value 100n -> 1µ; device iocene:C_402 -> iocene:C_603
- C30, C31, C39: value 10u -> 1µ; device iocene:C_805 -> iocene:C_603
- C33, C34, C35, C36, C44, C60, C61, C62, C63, C64, C65, C66, C69, C70, C79: device iocene:C_402 -> iocene:C_603
- C40: value 1u -> 1µ
- C42: value 10n -> 100n; device iocene:C_402 -> iocene:C_603
- C43: value 100p -> 100n; device iocene:C_402 -> iocene:C_603
- C45: value 22n -> 100n; device iocene:C_402 -> iocene:C_603
- C46: value 22n -> 100n
- C47: value 22n -> 1µ; device iocene:C_402 -> iocene:C_603
- C48, C49, C50, C83, C84: value 100n -> 1µ
- C52, C53, C54, C55: value 1µ -> 100n
- C57, C59, C72, C97: value 100n -> 10n
- C68: value 2.2u -> 100n
- C71: value 2.2u -> 1n; device iocene:C_603 -> iocene:C_402
- C73: value 18p -> 100n
- C74: value 18p -> 100n; device iocene:C_402 -> iocene:C_603
- C80: value 1n -> 100n; device iocene:C_402 -> iocene:C_603
- C86: value NC -> 100n; device iocene:C_402 -> iocene:C_603
- C87: value 470u -> 100n; device iocene:CPOL -> iocene:C_603
- C92: value 100n -> 10n; device iocene:C_805 -> iocene:C_402
- CON1: value M2 -> CON2_3.81
- CON10: value QEI3 -> M5; device iocene:CON5_2.54S -> iocene:CON2_3.81
- CON11: value QEI2 -> M2; device iocene:CON5_2.54S -> iocene:CON2_3.81
- CON12: value CON14 -> M4; device iocene:CON14 -> iocene:CON2_3.81
- CON13: value UART1 -> M0; device iocene:CON5_2.54S -> iocene:CON2_3.81
- CON14: value UART0 -> ESC0; device iocene:CON5_2.54S -> iocene:CON4_3.81
- CON15: value BALISE -> CON10_2_2.54; device iocene:CON5_2.54S -> iocene:CON10_2_2.54
- CON17: value CON10_2_2.54 -> ESC1; device iocene:CON10_2_2.54 -> iocene:CON4_3.81
- CON2: value TELEM -> CON2_3.81; device iocene:CON5_2.54S -> iocene:CON2_3.81
- CON28: value NC -> AN2; device iocene:USBUSB3140 -> iocene:CON3_SMT
- CON3: value M5 -> CON2_3.81
- CON4: value M3 -> CON2_3.81
- CON5: value M4 -> CON2_3.81
- CON6: value M0 -> CON2_3.81
- CON7: value M1 -> FPGApower
- CON8: value QEI1 -> M1; device iocene:CON5_2.54S -> iocene:CON2_3.81
- CON9: value QEI0 -> M3; device iocene:CON5_2.54S -> iocene:CON2_3.81
- D3: value SMP12A -> SMAJ51A; device iocene:ZENER -> iocene:ZENERDO214
- D4: value SMAJ51A -> LED_603; device iocene:ZENERDO214 -> iocene:LED_603
- IC1: value REF5025I -> ADS1258; device IMU:REF5025I -> IMU:ADS1258
- IC2: value REF5030I -> ADS1278; device IMU:REF5025I -> IMU:ADS1278"
- J1: value 0 -> NC; device iocene:JUMP_402 -> iocene:JUMP_603
- J10, J23, J8: device iocene:JUMP_603 -> iocene:JUMP_402
- J18: value (none) -> 0; device SparkFun-Connectors:M05X2NO_SILK -> iocene:JUMP_402
- J2, J30, J33: value 0 -> nc
- J20, J25, J31: value nc -> 0
- J24, J4, J6: device iocene:JUMP_402 -> iocene:JUMP_603
- J5: value 0 -> nc; device iocene:JUMP_402 -> iocene:JUMP_603
- J9: value nc -> 0; device iocene:JUMP_603 -> iocene:JUMP_402
- L10, L9: value SRN2512-R24M -> 600; device iocene:INDUCTANCE_2520 -> iocene:INDUCTANCE_603
- L8: value 600 -> SRN2512-R24M; device iocene:INDUCTANCE_603 -> iocene:INDUCTANCE_2520
- R1, R2: value 560 -> 100k
- R10: value 12.4k -> 560
- R100, R104, R106: value 100k -> 10k
- R101, R105: value 19k -> 10k
- R102, R103, R82, R84, R85, R86, R87, R89: value 1k -> 10k
- R11, R12, R13: value 10k -> 560
- R14, R5, R6, R7: value 10k -> 5k
- R15, R3: value 10k -> 100k
- R16: value 10k -> 32k
- R20: value 10k -> 19k
- R23: value 12k -> ULR15S-R0055FT2; device iocene:R_402 -> iocene:R_ULR15S-R0055FT2
- R24, R32: value 10k -> ULR15S-R0055FT2; device iocene:R_402 -> iocene:R_ULR15S-R0055FT2
- R26, R28, R30: value 10k -> 30k
- R35, R48, R54, R56, R63: value 0.01 -> 10k; device iocene:R_603 -> iocene:R_402
- R36: value 30k -> ULR15S-R0055FT2; device iocene:R_402 -> iocene:R_ULR15S-R0055FT2
- R37, R43, R44: value ULR15S-R0055FT2 -> 10k; device iocene:R_ULR15S-R0055FT2 -> iocene:R_402
- R39, R62, R71, R72, R73: value 10k -> 1k
- R4: value 330 -> 100k
- R40: value 30k -> 1k
- R41, R42: value 30k -> 10k
- R45, R52, R57, R65, R70, R78: value 10k -> 0.01; device iocene:R_402 -> iocene:R_603
- R50, R58, R61: value 0.01 -> 1k; device iocene:R_603 -> iocene:R_402
- R66: value 1M -> 10k
- R8: value 330 -> 5k
- R83, R88: value 1k -> 0.01; device iocene:R_402 -> iocene:R_603
- R9: value 1M -> 240
- R90: value 10k -> 1M
- R92: value 10k -> 330
- R94: value ULR15S-R0055FT2 -> 330; device iocene:R_ULR15S-R0055FT2 -> iocene:R_402
- R95: value 10k -> 12.4k
- R96: value ULR15S-R0055FT2 -> 12k; device iocene:R_ULR15S-R0055FT2 -> iocene:R_402
- R97: value 240 -> 10k
- R98: value 560 -> 1M
- R99: value 32k -> 10k
- U10: value LAN9514 -> DRV8432; device iocene:LAN9514 -> iocene:DRV84X2_DRV8432
- U13: value LP5900_2.2 -> INA240-A2; device iocene:REG_EN_LP5900 -> Texas Instruments_By_element14_Batch_1:INA240-TSSOP
- U14: value ESC_TURNIGY40A -> DRV8432; device iocene:ESC_TURNIGY40A -> iocene:DRV84X2_DRV8432
- U16: value ESC_CHINOI15A -> INA240-A2; device iocene:ESC_CHINOI15A -> Texas Instruments_By_element14_Batch_1:INA240-TSSOP
- U17: value TPS82130 -> ESC_TURNIGY40A; device iocene:TPS82130 -> iocene:ESC_TURNIGY40A
- U18: value TPS82130 -> INA240-A2; device iocene:TPS82130 -> Texas Instruments_By_element14_Batch_1:INA240-TSSOP
- U19: value TPS82130 -> ESC_CHINOI15A; device iocene:TPS82130 -> iocene:ESC_CHINOI15A
- U2: value OPA376 -> BUZZER; device iocene:OPA376 -> iocene:BUZZER
- U20: value SN74LV4052A_SO -> LAN9514; device iocene:SN74LV4052A_SO -> iocene:LAN9514
- U21: value BUZZER -> LGA22U; device iocene:BUZZER -> Gemicom:LGA22U
- U4: value ARDUINOR3-DIMENSION -> TPS82130; device adafruit:ARDUINOR3-DIMENSION -> iocene:TPS82130
- renumbered AN0 to CON20, AN1 to CON23, AN3 to CON33, AN4 to CON37, AN5 to CON42, AN6 to CON46, AN7 to CON50, C197 to C120, I2C0 to CON49, I2C1 to CON53, IO0 to CON22, IO1 to CON25, IO2 to CON30, IO3 to CON35, IO4 to CON39, IO5 to CON44, IO6 to CON48, IO7 to CON52, J121 to J37, J122 to J38, J123 to J41, J124 to J42, J125 to J45, J126 to J46, J127 to J35, J128 to J36, J129 to J39, J130 to J40, J131 to J43, J132 to J44, JP1_GPIO0 to CON57, JP7_GPIO1 to CON58, R110 to R25, R111 to R22, S0 to CON21, S1 to CON24, S2 to CON29, S3 to CON34, S4 to CON38, S5 to CON43, S6 to CON47, S7 to CON51, SPI0 to CON40, SPI1 to CON45, U$1 to U30, U$10 to U31, U$11 to U32, U$13 to K1, U$14 to U3, U$2 to U25, U$21 to U7, U$23 to U11, U$25 to U9, U$26 to U15, U$27 to U12, U$3 to U8, U$30 to K2, U$32 to K3, U$33 to K4, U$4 to U27, U$6 to U22, U$8 to U26, U$9 to U28, USB2 to CON54, USB3 to CON55, UW2 to Q2
Connections:
- removed net N$152: C86.P$2, CON28.VBUS, L14.2
- new net ADC_IN0: J47.2
- net 12V: now also C16.P$1, C2.+, C20.P$1, C24.P$1, CON1.2, CON36.4, J1.2, R1.P$1, U4.EN, U4.VI, U5.EN, U5.VI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; no longer C184.P$1, C188.P$1, C30.P$1, C89.+, CON15.4, J133.2, LIPO_ELEC.2, R112.P$1, U17.EN, U17.VI, U18.EN, U18.VI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
- net 24V: now also C11.P$1, C12.+, C33.P$2, C34.P$2, C35.P$2, C36.P$2, C77.P$2, C78.P$2, C79.P$2, C80.P$2, CON3.2, D3.C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; no longer C114.P$2, C115.P$2, C116.P$2, C117.P$2, C129.P$2, C130.P$2, C131.P$2, C132.P$2, C141.+, C92.P$1, D4.C, J25.1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
- net 3V3: now also C138.P$2, C139.P$2, C140.P$2, C141.P$2, C142.P$2, C17.P$1, C18.+, D9.A, L9.1, R15.P$1, R89.P$2, R91.P$2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; no longer C156.+, C31.P$1, C58.P$2, C59.P$2, C60.P$2, C61.P$2, C62.P$2, D11.A, L8.1, R100.P$1, R24.P$2, R3.P$2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
- net 5V: now also C103.P$2, C109.P$2, C118.P$2, C125.P$2, C149.P$2, C152.P$2, C159.P$2, C161.P$2, C165.P$2, C172.P$2, C173.P$2, C174.P$2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; no longer AN2.2, C134.P$2, C139.P$2, C140.P$2, C154.P$2, C155.P$2, C158.P$2, C160.P$2, C166.P$2, C170.P$2, C185.P$1, C186.+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
- net A12V: now also C13.P$1, C29.P$2, C30.P$2, C31.P$2, C32.P$2, C38.P$2, C39.P$2, C40.P$2, C41.P$2, C47.P$2, C48.P$2, C49.P$2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; no longer C108.P$2, C109.P$2, C110.P$2, C111.P$2, C124.P$2, C125.P$2, C126.P$2, C127.P$2, C28.P$1, C52.P$2, C53.P$2, C54.P$2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
- net A5V: now also C14.P$1, C15.+, C94.P$1, C99.P$1, CON15.2, J26.1, J27.1, R12.P$1, R2.P$1; no longer C172.P$1, C178.P$1, C181.+, C182.P$1, CON17.2, J28.1, J29.1, R114.P$1, R98.P$1
- net AD0_CLK: now also IC2.CLK; no longer UV1.CLK
- net AD0_DRDY: now also IC2.DRDY/; no longer UV1.DRDY/
- net AD0_MISO: now also IC2.DOUT1; no longer UV1.DOUT1
- net AD0_SCLK: now also IC2.SCLK; no longer UV1.SCLK
- net AD0_SYNC: now also IC2.SYNC; no longer UV1.SYNC
- net AD0_VREF: now also C171.P$2, C180.P$1, C57.P$2, C59.P$2, C72.P$2, CON16.10, IC2.AINN2, IC2.AINN3, IC2.AINN4, IC2.AINN5, IC2.AINN6, IC2.AINN7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; no longer C121.P$2, C135.P$2, C167.P$2, C168.P$1, C193.P$2, CON17.10, J22.2, J24.1, U$22.REF1, U$22.REF2, UV1.AINN2, UV1.AINN3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
- net AD0_VREF*: now also C92.P$2, C97.P$2, CON15.10, U16.REF1, U16.REF2, U18.REF1, U18.REF2; no longer C174.P$2, C180.P$2, CON16.10, U$31.REF1, U$31.REF2, U$34.REF1, U$34.REF2
- net AD1_DRDY: now also IC1.DRDY, U29.D11; no longer U4.D11, UW1.DRDY
- net AD1_M: now also IC1.MUXOUTP, R97.P$1; no longer R65.P$1, UW1.MUXOUTP
- net AD1_MISO: now also IC1.DOUT, U29.D12; no longer U4.D12, UW1.DOUT
- net AD1_MOSI: now also IC1.DIN, U29.D13; no longer U4.D13, UW1.DIN
- net AD1_P: now also C178.P$2, IC1.ADCINP, R98.P$2, U24.OUT; no longer C43.P$2, R66.P$2, U2.OUT, UW1.ADCINP
- net AD1_RST: now also IC1.RESET, U29.SCL; no longer U4.SCL, UW1.RESET
- net AD1_SCLK: now also IC1.SCLK, U29.SDA; no longer U4.SDA, UW1.SCLK
- net AD1_SS: now also IC1.CS, U29.D10; no longer U4.D10, UW1.CS
- net AD1_V: now also C176.P$1, C177.P$2, IC1.VREFP, J31.2; no longer C39.P$1, C42.P$2, J21.2, UW1.VREFP
- net ADC_IN1: now also J47.3; no longer J18.3
- net ADC_IN2: now also J47.4; no longer J18.4
- net ADC_IN3: now also J47.5; no longer J18.5
- net ADC_IN4: now also J47.6; no longer J18.6
- net ADC_IN5: now also J47.7; no longer J18.7
- net ADC_IN6: now also J47.8; no longer J18.8
- net ADC_IN7: now also J47.9; no longer J18.9
- net ADC_VCC: now also J47.1; no longer J18.1
- net AN0: now also C100.P$2, IC1.AIN7, R41.P$2, R43.P$1; no longer C2.P$2, R21.P$1, R67.P$2, UW1.AIN7
- net AN1: now also C106.P$2, IC1.AIN6, R46.P$2, R48.P$1; no longer C3.P$2, R20.P$1, R68.P$2, UW1.AIN6
- net AN2: now also C112.P$2, IC1.AIN5, R53.P$2, R55.P$1; no longer C4.P$2, R69.P$1, R70.P$2, UW1.AIN5
- net AN3: now also C115.P$2, IC1.AIN4, R59.P$2, R63.P$1; no longer C5.P$2, R71.P$1, R72.P$2, UW1.AIN4
- net AN4: now also C122.P$2, IC1.AIN3, R66.P$2, R68.P$1; no longer C6.P$2, R73.P$1, R74.P$2, UW1.AIN3
- net AN5: now also C129.P$2, IC1.AIN2, R74.P$2, R76.P$1; no longer C7.P$2, R75.P$1, R76.P$2, UW1.AIN2
- net AN6: now also C132.P$2, IC1.AIN1, R79.P$2, R81.P$1; no longer C8.P$2, R77.P$1, R78.P$2, UW1.AIN1
- net AN7: now also C135.P$2, IC1.AIN0, R84.P$2, R86.P$1; no longer C9.P$2, R79.P$1, R80.P$2, UW1.AIN0
- net ARDUINO_A0: now also U29.A0; no longer U4.A0
- net ARDUINO_A1: now also U29.A1; no longer U4.A1
- net ARDUINO_A2: now also U29.A2; no longer U4.A2
- net ARDUINO_A3: now also U29.A3; no longer U4.A3
- net ARDUINO_A4: now also U29.A4/SDA; no longer U4.A4/SDA
- net ARDUINO_A5: now also U29.A5/SCL; no longer U4.A5/SCL
- net BALISE: now also U29.D3; no longer U4.D3
- net BALISE°: now also CON36.5; no longer CON15.5
- net BUZZER: now also U29.D8; no longer U4.D8
- net BUZZER°: now also T1.G; no longer T3.G
- net D3V3: now also C160.P$2, C167.P$2, C181.P$2, C183.P$2, C185.P$2, C187.P$2, C189.P$2, C191.P$2, C193.P$2, C3.P$1, IC1.DVDD, IC1.PWDN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; no longer C10.P$2, C12.P$2, C137.P$2, C150.P$2, C157.P$2, C161.P$2, C21.P$2, C210.P$1, C23.P$2, C25.P$2, J120.2, J20.2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
- net DM2: now also U20.USBDM3; no longer U10.USBDM2
- net DM3: now also U20.USBDM4; no longer U10.USBDM3
- net DP2: now also U20.USBDP3; no longer U10.USBDP2
- net DP3: now also U20.USBDP4; no longer U10.USBDP3
- net ESC0_CS: now also C96.P$2, CON16.7, IC2.AINP3; no longer C179.P$2, CON17.7, UV1.AINP3
- net ESC0_CS*: now also CON15.7, R35.P$2; no longer CON16.7, R93.P$2
- net ESC0_DIR: now also U29.D5; no longer U4.D5
- net ESC0_DIR°: now also CON16.3; no longer CON17.3
- net ESC0_DIR°*: now also CON15.3, T2.G; no longer CON16.3, T1.G
- net ESC0_PWM: now also U29.D4; no longer U4.D4
- net ESC0_PWM°: now also CON16.5; no longer CON17.5
- net ESC0_PWM°*: now also CON15.5, U17.PWM; no longer CON16.5, U14.PWM
- net ESC1_CS: now also C95.P$2, CON16.8, IC2.AINP2; no longer C173.P$2, CON17.8, UV1.AINP2
- net ESC1_CS*: now also CON15.8, R37.P$2; no longer CON16.8, R95.P$2
- net ESC1_DIR: now also U29.D6; no longer U4.D6
- net ESC1_DIR°: now also CON16.4; no longer CON17.4
- net ESC1_DIR°*: now also CON15.4, T3.G; no longer CON16.4, T2.G
- net ESC1_PWM: now also U29.D7; no longer U4.D7
- net ESC1_PWM°: now also CON16.1; no longer CON17.1
- net ESC1_PWM°*: now also CON15.1, U19.PWM; no longer CON16.1, U16.PWM
- net ESC_PWR: now also C91.+, J24.2, R36.P$2, R38.P$2, U16.IN-, U18.IN+; no longer C87.+, J23.2, R94.P$2, R96.P$2, U$31.IN-, U$34.IN+
- net GND: now also C10.P$2, C102.P$1, C103.P$1, C104.P$1, C105.P$1, C106.P$1, C107.P$1, C11.P$2, C113.P$1, C12.-, C122.P$1, C123.P$1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; no longer AN2.1, C10.P$1, C11.P$1, C12.P$1, C13.P$1, C14.P$1, C141.-, C15.P$1, C156.-, C16.P$1, C168.P$2, C169.P$2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
- net IO0°: now also C102.P$2, R42.P$2; no longer C142.P$2, R26.P$2
- net IO1°: now also C108.P$2, R47.P$2; no longer C143.P$2, R28.P$2
- net IO2°: now also C114.P$2, R54.P$2; no longer C144.P$2, R30.P$2
- net IO3°: now also C117.P$2, R60.P$2; no longer C145.P$2, R32.P$2
- net IO4°: now also C124.P$2, R67.P$2; no longer C146.P$2, R34.P$2
- net IO5°: now also C131.P$2, R75.P$2; no longer C147.P$2, R52.P$2
- net IO6°: now also C134.P$2, R80.P$2; no longer C148.P$2, R90.P$2
- net IO7°: now also C137.P$2, R85.P$2; no longer C149.P$2, R92.P$2
- net LAN_3V3: now also C143.P$2, C144.P$2, C145.P$2, C146.P$2, C147.P$2, C148.P$2, L9.2, U20.VDD33A, U20.VDD33A@1, U20.VDD33A@2, U20.VDD33A@3, U20.VDD33A@4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; no longer C63.P$2, C64.P$2, C65.P$2, C66.P$2, C67.P$2, C68.P$2, L8.2, U10.VDD33A, U10.VDD33A@1, U10.VDD33A@2, U10.VDD33A@3, U10.VDD33A@4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
- net LEDA: now also R10.P$1; no longer R2.P$1
- net LEDB: now also R11.P$1; no longer R1.P$1
- net LOW_VOLTAGE: now also C4.P$1, IC2.AINP1, U1.X; no longer C209.P$1, U20.X, UV1.AINP1
- net LV_MUXA: now also U1.A; no longer U20.A
- net LV_MUXB: now also U1.B; no longer U20.B
- net M0_CS: now also C90.P$2, IC2.AINP7, R34.P$2; no longer C119.P$2, R45.P$2, UV1.AINP7
- net M0_FAULT: now also U14.FAULT, U14.OT; no longer U$24.FAULT, U$24.OT
- net M0_PWMA: now also U14.PWMA; no longer U$24.PWMA
- net M0_PWMB: now also U14.PWMB; no longer U$24.PWMB
- net M1_CS: now also C71.P$2, IC2.AINP8, R27.P$2; no longer C133.P$2, R46.P$2, UV1.AINP8
- net M23_FAULT: now also U10.FAULT, U10.OT; no longer U$20.FAULT, U$20.OT
- net M2_CS: now also C76.P$2, IC2.AINP6, R31.P$2; no longer C80.P$2, R39.P$2, UV1.AINP6
- net M2_PWMA: now also U10.PWMC; no longer U$20.PWMC
- net M2_PWMB: now also U10.PWMD; no longer U$20.PWMD
- net M3_CS: now also C56.P$2, IC2.AINP5, R21.P$2; no longer C118.P$2, R59.P$2, UV1.AINP5
- net M3_PWMA: now also U10.PWMA; no longer U$20.PWMA
- net M3_PWMB: now also U10.PWMB; no longer U$20.PWMB
- net M4_CS: now also C58.P$2, IC2.AINP4; no longer C192.P$2, UV1.AINP4
- net N$1: now also CON3.1, CON4.2; no longer LIPO_MOTEUR.1, LIPO_MOTEUR1.2
- net N$10: now also C68.P$1, U10.BSTC; no longer C50.P$1, U$20.BSTC
- net N$100: now also C88.P$1, U14.BSTD; no longer C107.P$1, U$24.BSTD
- net N$101: now also C87.P$1, U14.BSTC; no longer C106.P$1, U$24.BSTC
- net N$102: now also C86.P$1, U14.BSTB; no longer C104.P$1, U$24.BSTB
- net N$103: now also C85.P$2, L5.2, U14.OUTA; no longer C102.P$2, L2.2, U$24.OUTA
- net N$104: now also C86.P$2, L6.2, U14.OUTB; no longer C104.P$2, L4.2, U$24.OUTB
- net N$105: now also C87.P$2, L7.2, U14.OUTC; no longer C106.P$2, L3.2, U$24.OUTC
- net N$106: now also C88.P$2, L8.2, U14.OUTD; no longer C107.P$2, L7.2, U$24.OUTD
- net N$11: now also CON13.2, R32.P$2; no longer CON6.2, R44.P$2
- net N$110: now also C157.P$2, C158.P$2, L10.2, U20.VDD18USBPLL; no longer C18.P$2, C57.P$2, L13.2, U10.VDD18USBPLL
- net N$111: now also C153.P$2, C154.P$2, C155.P$2, U20.VDD18CORE, U20.VDD18CORE@1; no longer C69.P$2, C70.P$2, C71.P$2, U10.VDD18CORE, U10.VDD18CORE@1
- net N$112: now also C156.P$2, L10.1, U20.VDD18ETHPLL; no longer C72.P$2, L13.1, U10.VDD18ETHPLL
- net N$113: now also R95.P$2, U20.EXRES; no longer R10.P$2, U10.EXRES
- net N$114: now also C89.P$2, J20.1, J21.1, J23.1, U14.VCAP; no longer C112.P$2, J11.1, J12.1, J17.1, U$24.VCAP
- net N$115: now also R33.P$1, U14.OC_ADJ; no longer R41.P$1, U$24.OC_ADJ
- net N$116: now also C55.P$1; no longer C105.P$1
- net N$117: now also J21.2, U14.RST_CD; no longer J11.2, U$24.RST_CD
- net N$118: now also J22.2, U14.M1; no longer J13.2, U$24.M1
- net N$119: now also J23.2, U14.M2; no longer J12.2, U$24.M2
- net N$12: now also C64.P$1, U10.BSTB; no longer C49.P$1, U$20.BSTB
- net N$120: now also C65.P$1; no longer C123.P$1
- net N$121: now also R34.P$1; no longer R45.P$1
- net N$123: now also C62.P$1; no longer C122.P$1
- net N$124: now also L8.1, R32.P$1; no longer L3.1, R44.P$1
- net N$125: now also C60.P$1; no longer C113.P$1
- net N$126: now also CON13.1, L5.1, L6.1; no longer CON6.1, L2.1, L4.1
- net N$127: now also C55.P$2, L1.2; no longer C105.P$2, L9.2
- net N$128: now also C60.P$2, L2.2; no longer C113.P$2, L11.2
- net N$129: now also C62.P$2, L3.2; no longer C122.P$2, L10.2
- net N$13: now also CON10.1; no longer CON3.1
- net N$130: now also C65.P$2, L4.2; no longer C123.P$2, L12.2
- net N$131: now also C67.P$2, J11.1, J8.1, J9.1; no longer C128.P$2, J14.1, J15.1, J32.1
- net N$132: now also R26.P$1; no longer R42.P$1
- net N$133: now also J9.2; no longer J14.2
- net N$134: now also J10.2; no longer J16.2
- net N$135: now also J11.2; no longer J15.2
- net N$136: now also R27.P$1; no longer R46.P$1
- net N$138: now also L3.1, L4.1, R24.P$1; no longer L10.1, L12.1, R43.P$1
- net N$139: now also CON8.1, L1.1, L2.1; no longer CON7.1, L11.1, L9.1
- net N$14: now also C61.P$2, R23.P$1, U10.OUTA; no longer C48.P$2, R37.P$1, U$20.OUTA
- net N$149: now also R96.P$2, U20.USBRBIAS; no longer R23.P$2, U10.USBRBIAS
- net N$15: now also C74.P$2, CON12.2; no longer C88.P$2, CON5.2
- net N$150: now also C151.P$2, R90.P$1, U20.XO; no longer C74.P$2, R9.P$1, U10.XO
- net N$151: now also CON56.2, U20.USBDP0; no longer CON28.D+, U10.USBDP0
- net N$153: now also CON56.3, U20.USBDM0; no longer CON28.D-, U10.USBDM0
- net N$154: now also R89.P$1, U20.NRESET; no longer R24.P$1, U10.NRESET
- net N$155: now also C150.P$2, R90.P$2, U20.XI; no longer C73.P$2, R9.P$2, U10.XI
- net N$156: now also R85.P$1; no longer R92.P$1
- net N$157: now also C19.P$1, U4.SS; no longer C183.P$1, U17.SS
- net N$158: now also R42.P$1; no longer R26.P$1
- net N$159: now also R47.P$1; no longer R28.P$1
- net N$16: now also C64.P$2, CON9.2, U10.OUTB; no longer C49.P$2, CON4.2, U$20.OUTB
- net N$160: now also R54.P$1; no longer R30.P$1
- net N$161: now also R60.P$1; no longer R32.P$1
- net N$162: now also R67.P$1; no longer R34.P$1
- net N$163: now also R75.P$1; no longer R52.P$1
- net N$164: now also R80.P$1; no longer R90.P$1
- net N$166: now also IC2.VCOM, J30.2; no longer J24.2, UV1.VCOM
- net N$167: now also IC2.MODE0, J28.1, J29.2; no longer J19.2, J20.1, UV1.MODE0
- net N$168: now also C179.P$1, IC4.TRIM; no longer C169.P$1, IC1.TRIM
- net N$169: now also C166.P$2, IC2.DVDD, U23.VO; no longer C165.P$2, U13.VO, UV1.DVDD
- net N$17: now also J20.2, U14.RST_AB; no longer J17.2, U$24.RST_AB
- net N$170: now also IC4.VOUT, J32.1; no longer IC1.VOUT, J22.1
- net N$171: now also CON41.4, R71.P$2; no longer CON11.4, R85.P$2
- net N$172: now also CON41.3, R72.P$2; no longer CON11.3, R86.P$2
- net N$173: now also CON41.2, R73.P$2; no longer CON11.2, R87.P$2
- net N$174: now also CON32.4, R58.P$2; no longer CON10.4, R82.P$2
- net N$175: now also CON32.3, R61.P$2; no longer CON10.3, R83.P$2
- net N$176: now also CON32.2, R62.P$2; no longer CON10.2, R84.P$2
- net N$177: now also U17.W; no longer U14.W
- net N$178: now also U17.U; no longer U14.U
- net N$18: now also J16.2, U10.M1; no longer J3.2, U$20.M1
- net N$180: now also CON14.2; no longer ESC0.2
- net N$181: now also CON14.3; no longer ESC0.3
- net N$182: now also CON14.1, U17.V; no longer ESC0.1, U14.V
- net N$184: now also R35.P$1, U16.OUT; no longer R93.P$1, U$31.OUT
- net N$185: now also R36.P$1, U16.IN+, U17.PWR; no longer R94.P$1, U$31.IN+, U14.PWR
- net N$187: now also J27.2, U19.VCC; no longer J28.2, U16.VCC
- net N$188: now also J26.2, U17.VCC; no longer J29.2, U14.VCC
- net N$189: now also U19.W; no longer U16.W
- net N$19: now also J8.2; no longer J32.2
- net N$190: now also U19.U; no longer U16.U
- net N$191: now also CON17.2; no longer ESC1.2
- net N$192: now also CON17.3; no longer ESC1.3
- net N$193: now also CON17.1, U19.V; no longer ESC1.1, U16.V
- net N$195: now also R37.P$1, U18.OUT; no longer R95.P$1, U$34.OUT
- net N$196: now also R38.P$1, U18.IN-, U19.PWR; no longer R96.P$1, U$34.IN-, U16.PWR
- net N$198: now also R17.P$2, R18.P$1, U5.ADJ; no longer R101.P$1, R104.P$2, U18.ADJ
- net N$199: now also C23.P$1, U5.SS; no longer C187.P$1, U18.SS
- net N$20: now also J12.2, U10.RST_AB; no longer J33.2, U$20.RST_AB
- net N$200: now also R9.P$1; no longer R97.P$1
- net N$201: now also R19.P$2, R20.P$1, U6.ADJ; no longer R105.P$1, R106.P$2, U19.ADJ
- net N$202: now also C27.P$1, U6.SS; no longer C191.P$1, U19.SS
- net N$204: now also D7.A, R13.P$2; no longer D6.A, R108.P$2
- net N$205: now also D8.A, R14.P$2; no longer D7.A, R109.P$2
- net N$206: now also C25.P$1, C26.+, CON7.2, R19.P$1, U6.VO; no longer C189.P$1, C190.+, FPGA_POWER.2, R106.P$1, U19.VO
- net N$207: now also C7.P$1, R1.P$2, R5.P$1, U1.X3; no longer C195.P$1, R112.P$2, R113.P$1, U20.X3
- net N$21: now also R52.P$1; no longer R48.P$1
- net N$210: now also C10.P$1, R4.P$2, R8.P$1, U1.X0; no longer C208.P$1, R116.P$2, R117.P$1, U20.X0
- net N$211: now also C8.P$1, R2.P$2, R6.P$1, U1.X2; no longer C206.P$1, R114.P$2, R119.P$1, U20.X2
- net N$212: now also C9.P$1, R3.P$2, R7.P$1, U1.X1; no longer C207.P$1, R115.P$2, R118.P$1, U20.X1
- net N$213: now also T1.D, U2.-; no longer T3.D, U21.-
- net N$214: now also J2.2, J3.2, U2.+; no longer J30.2, J31.2, U21.+
- net N$22: now also J14.2; no longer J34.2
- net N$23: now also R56.P$2, R57.P$1; no longer R50.P$1, R53.P$2
- net N$25: now also R97.P$2, R98.P$1, U24.-; no longer R65.P$2, R66.P$1, U2.-
- net N$27: now also R84.P$1; no longer R80.P$1
- net N$28: now also R41.P$1; no longer R67.P$1
- net N$3: now also CON4.1, CON5.2; no longer LIPO_MOTEUR1.1, LIPO_MOTEUR2.2
- net N$30: now also R46.P$1; no longer R68.P$1
- net N$31: now also C182.P$2, J33.1, J34.1; no longer C13.P$2, J119.1, J120.1
- net N$32: now also CON28.3, R53.P$1; no longer AN2.3, R70.P$1
- net N$33: now also R59.P$1; no longer R72.P$1
- net N$34: now also R66.P$1; no longer R74.P$1
- net N$35: now also C186.P$2, R100.P$2, R99.P$2; no longer C11.P$2, R5.P$2, R6.P$2
- net N$36: now also C190.P$2, R103.P$2, R104.P$2; no longer C14.P$2, R13.P$2, R14.P$2
- net N$37: now also C194.P$2; no longer C15.P$2
- net N$38: now also C184.P$2; no longer C16.P$2
- net N$39: now also C188.P$2; no longer C17.P$2
- net N$4: now also CON5.1, CON6.2; no longer LIPO_MOTEUR2.1, LIPO_MOTEUR3.2
- net N$40: now also C192.P$2; no longer C19.P$2
- net N$41: now also D6.A, R12.P$2; no longer D5.A, R98.P$2
- net N$42: now also R15.P$2, R16.P$1, U4.ADJ; no longer R100.P$2, R99.P$1, U17.ADJ
- net N$43: now also R64.P$2, R65.P$1; no longer R54.P$1, R55.P$2
- net N$44: now also R69.P$2, R70.P$1; no longer R56.P$1, R57.P$2
- net N$45: now also R77.P$2, R78.P$1; no longer R58.P$1, R60.P$2
- net N$46: now also J17.2, U10.M2; no longer J2.2, U$20.M2
- net N$47: now also R82.P$2, R83.P$1; no longer R61.P$1, R62.P$2
- net N$48: now also R87.P$2, R88.P$1; no longer R63.P$1, R64.P$2
- net N$49: now also C168.P$2, IC1.XTAL1; no longer C46.P$2, UW1.XTAL1
- net N$5: now also J13.2, U10.RST_CD; no longer J1.2, U$20.RST_CD
- net N$50: now also C175.P$1, IC3.TRIM; no longer C40.P$1, IC2.TRIM
- net N$51: now also IC3.VOUT, J31.1; no longer IC2.VOUT, J21.1
- net N$52: now also T3.D; no longer T2.D
- net N$53: now also C170.P$2, IC1.PLLCAP; no longer C45.P$2, UW1.PLLCAP
- net N$54: now also C169.P$2, IC1.XTAL2; no longer C47.P$2, UW1.XTAL2
- net N$55: now also C68.P$2, CON11.1, U10.OUTC; no longer C50.P$2, CON1.1, U$20.OUTC
- net N$56: now also C70.P$2, R29.P$1, U10.OUTD, U13.IN-; no longer C51.P$2, R38.P$1, U$20.OUTD, U$22.IN-
- net N$57: now also C73.P$2, J12.1, J13.1, U10.VCAP; no longer C56.P$2, J1.1, J33.1, U$20.VCAP
- net N$58: now also R74.P$1; no longer R76.P$1
- net N$59: now also R79.P$1; no longer R78.P$1
- net N$6: now also R44.P$2, R45.P$1; no longer R35.P$1, R47.P$2
- net N$60: now also CON9.1, R23.P$2; no longer CON4.1, R37.P$2
- net N$61: now also D5.A, R11.P$2; no longer D8.A, R1.P$2
- net N$62: now also R28.P$1, U10.OC_ADJ; no longer R36.P$1, U$20.OC_ADJ
- net N$63: now also T2.D; no longer T1.D
- net N$64: now also D4.A, R10.P$2; no longer D9.A, R2.P$2
- net N$65: now also R21.P$1; no longer R59.P$1
- net N$66: now also R94.P$2; no longer R4.P$2
- net N$67: now also D9.C, R92.P$2; no longer D11.C, R8.P$2
- net N$7: now also C61.P$1, U10.BSTA; no longer C48.P$1, U$20.BSTA
- net N$76: now also CON11.2, R29.P$2, U13.IN+; no longer CON1.2, R38.P$2, U$22.IN+
- net N$77: now also C63.P$1; no longer C83.P$1
- net N$78: now also C74.P$1; no longer C88.P$1
- net N$79: now also C69.P$1; no longer C85.P$1
- net N$8: now also C70.P$1, U10.BSTD; no longer C51.P$1, U$20.BSTD
- net N$80: now also C66.P$1; no longer C84.P$1
- net N$81: now also C63.P$2; no longer C83.P$2
- net N$82: now also C66.P$2, CON10.2; no longer C84.P$2, CON3.2
- net N$83: now also C69.P$2, CON12.1; no longer C85.P$2, CON5.1
- net N$85: now also C75.P$2, J14.1, J15.1; no longer C97.P$2, J34.1, J4.1
- net N$86: now also R30.P$1; no longer R40.P$1
- net N$87: now also C42.P$2, C43.P$2, C44.P$2, C45.P$2, J4.2, J5.2, U10.VDDA, U10.VDDB, U10.VDDC, U10.VDDD; no longer C75.P$2, C76.P$2, C77.P$2, C78.P$2, J7.2, J8.2, U$20.VDDA, U$20.VDDB, U$20.VDDC, U$20.VDDD
- net N$88: now also J15.2; no longer J4.2
- net N$89: now also R31.P$1, U13.OUT; no longer R39.P$1, U$22.OUT
- net N$9: now also CON8.2, R24.P$2; no longer CON7.2, R43.P$2
- net N$90: now also J18.2; no longer J6.2
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
Commit message: Routage ok
Parts:
- added C195: 100n, iocene:C_402
- added CON60: USB3, iocene:USB_A
- added J48, J49: NC, iocene:JUMP_402
- CON1: value CON2_3.81 -> ELEC
- CON13: value M0 -> M1
- CON2: value CON2_3.81 -> SERVO
- CON3, CON4, CON5, CON6: value CON2_3.81 -> LIPO_MOT
- CON56: value CON3_2.54S -> USBfpga
- CON57: value CON40_2.54 -> FPGA_GPIO0
- CON58: value CON40_2.54 -> FPGA_GPIO1
- CON59: value CON14 -> FPGA_LTC
- CON8: value M1 -> M0
- J47: value (none) -> FPGA_ADC
- U29: value ARDUINOR3-DIMENSION -> FPGA_ARDUINO
Connections:
- new net N$2: CON60.D-, J48.1
- new net N$24: CON60.D+, J49.1
- net 5V: now also C195.P$2, CON60.VBUS
- net GND: now also C195.P$1, CON60.GND, CON60.GND@2
- net M0_CS: now also C71.P$2, IC2.AINP8, R27.P$2; no longer C90.P$2, IC2.AINP7, R34.P$2
- net M0_FAULT: now also CON57.27, U9.FAULT, U9.OT; no longer CON57.24, U14.FAULT, U14.OT
- net M0_PWMA: now also CON57.28, U9.PWMA; no longer CON57.25, U14.PWMA
- net M0_PWMB: now also CON57.32, U9.PWMB; no longer CON57.26, U14.PWMB
- net M1_CS: now also C90.P$2, IC2.AINP7, R34.P$2; no longer C71.P$2, IC2.AINP8, R27.P$2
- net M1_FAULT: now also CON57.24, U14.FAULT, U14.OT; no longer CON57.27, U9.FAULT, U9.OT
- net M1_PWMA: now also CON57.25, U14.PWMA; no longer CON57.28, U9.PWMA
- net M1_PWMB: now also CON57.26, U14.PWMB; no longer CON57.32, U9.PWMB
- net WIFI1_DM: now also J48.2
- net WIFI1_DP: now also J49.2
Other:
- moved on the sheet: D10, D9, R91, R92, R93, R94
