File: hardware/expansion_board_V0/expansion_board_V0.sch (EAGLE design)
At the start: 501 parts, among them CON1 ELEC, CON10 M5, CON11 M2, CON12 M4, CON13 M1, CON14 ESC0, CON15 CON10_2_2.54, CON16 CON10_2_2.54, CON17 ESC1, CON18 UART0, CON19 QEI1, CON2 SERVO, CON20 AN0, CON21 S0, CON22 IO0, CON23 AN1, CON24 S1, CON25 IO1, CON26 UART1, CON27 QEI0, CON28 AN2, CON29 S2, CON3 LIPO_MOT, CON30 IO2, CON31 TELEM, CON32 QEI3, CON33 AN3, CON34 S3, CON35 IO3, CON36 BALISE, CON37 AN4, CON38 S4, CON39 IO4, CON4 LIPO_MOT, CON40 SPI0, CON41 QEI2, CON42 AN5, CON43 S5, CON44 IO5, CON45 SPI1, CON46 AN6, CON47 S6, CON48 IO6, CON49 I2C0, CON5 LIPO_MOT, CON50 AN7, CON51 S7, CON52 IO7, CON53 I2C1, CON54 USB2, CON55 USB3, CON56 USBfpga, CON57 FPGA_GPIO0, CON58 FPGA_GPIO1, CON59 FPGA_LTC, CON6 LIPO_MOT, CON60 USB3, CON61 CON5_2.54S, CON62 CON5_2.54S, CON63 CON5_2.54S, CON64 CON5_2.54S, CON7 FPGApower, CON8 M0, CON9 M3, IC1 ADS1258, IC2 ADS1278, IC3 REF5030I, IC4 REF5025I, J1 NC, J10 0, J11 0, J12 0, J13 0, J14 0, J15 0, J16 0, J17 0, J18 0, J19 0, J2 nc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

Commit message: elec ok
Parts:
- C108: value 100n -> NC
- C117: value nc -> 100n
- C119, C120, C121, C126, C127, C128: value 1n -> 100p
- C56, C58, C71, C76, C90, C95, C96: value 1n -> 100n
- R1, R2, R3: value 100k -> 3.3k
- R21, R22, R27, R31, R34, R35, R37: value 10k -> 100
- R4: value 100k -> 33k
- R47: value 1k -> 33
- R5, R6, R7: value 5k -> 1k
- R58, R61, R62, R71, R72, R73: value 1k -> 100
- R60: value 560 -> 1k
- R8: value 5k -> 3.3k
- R80, R85: value 560 -> 33
