File: hardware/expansion_board_V0/IMU board.sch (EAGLE design)
At the start: 499 parts, among them CON1 ELEC, CON10 M5, CON11 M2, CON12 M4, CON13 M1, CON14 ESC0, CON15 CON10_2_2.54, CON16 CON10_2_2.54, CON17 ESC1, CON18 UART0, CON19 QEI1, CON2 SERVO, CON20 AN0, CON21 S0, CON22 IO0, CON23 AN1, CON24 S1, CON25 IO1, CON26 UART1, CON27 QEI0, CON28 AN2, CON29 S2, CON3 LIPO_MOT, CON30 IO2, CON31 TELEM, CON32 QEI3, CON33 AN3, CON34 S3, CON35 IO3, CON36 BALISE, CON37 AN4, CON38 S4, CON39 IO4, CON4 LIPO_MOT, CON40 SPI0, CON41 QEI2, CON42 AN5, CON43 S5, CON44 IO5, CON45 SPI1, CON46 AN6, CON47 S6, CON48 IO6, CON49 I2C0, CON5 LIPO_MOT, CON50 AN7, CON51 S7, CON52 IO7, CON53 I2C1, CON54 USB2, CON55 USB3, CON56 USBfpga, CON57 FPGA_GPIO0, CON58 FPGA_GPIO1, CON59 FPGA_LTC, CON6 LIPO_MOT, CON60 USB3, CON61 CON5_2.54S, CON62 CON5_2.54S, CON63 CON5_2.54S, CON64 CON5_2.54S, CON7 FPGApower, CON8 M0, CON9 M3, IC1 ADS1258, IC2 ADS1278, IC3 REF5030I, IC4 REF5025I, J1 NC, J10 0, J11 0, J12 0, J13 0, J14 0, J15 0, J16 0, J17 0, J18 0, J19 0, J2 nc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

Commit message: -
Parts:
- removed R110: 10k, iocene:R_402
- removed U39: TCA6408A, iocene:I2C_EXPTCA6408A
- removed U40: LP5900SD-2.8, iocene:REG_EN_LP5900
- added C200: 10n, iocene:C_402
- added C201, C211, C212, C213, C214, C215: 100n, iocene:C_402
- added C202, C203, C204, C205, C206, C207, C208, C209, C210: 2.2u, iocene:C_603
- added CON65: IMU_UART, iocene:CON3_2.54S
- added CON68: SPI0, iocene:CON6_2.54S
- added D11: LED_603, iocene:LED_603
- added J52, J53, J54, J55: 0, iocene:JUMP_402
- added U$1: STM32F4R_64PIN_FOXCAR, stm32f4:STM32F4R_64PIN_FOXCAR
- C196, C199: value 2u -> 100n; device iocene:C_603 -> iocene:C_402
- CON63: value CON5_2.54S -> USB2; device iocene:CON5_2.54S -> iocene:USB_A
- CON64: value CON5_2.54S -> SPI0; device iocene:CON5_2.54S -> iocene:CON6_2.54S
- R109: value 10k -> 560
- U36: value VL6180X -> MPU-9250; device iocene:VL6180X -> 9dof-devboard-temp:MPU-9250
Connections:
- removed net N$75: CON63.4, CON64.4, U36.SCL, U39.SCL
- removed net N$94: CON64.3, R110.P$1, U39.RST
- removed net N$95: CON63.3, U39.P7
- removed net N$97: R109.P$1, U36.RST, U39.P2
- new net D3/FSYNC: U$1.PC7, U36.FSYNC
- new net D4/INT: U$1.PC6, U36.INT
- new net IMU_/CS: J55.1, U$1.PA4, U36.!CS
- new net IMU_CLK: J54.1, U$1.PA5, U36.SCL/SCLK
- new net IMU_DM: CON63.D-, U$1.PA11
- new net IMU_DP: CON63.D+, U$1.PA12
- new net IMU_MISO: J52.1, U$1.PA6, U36.AD0/SDO
- new net IMU_MOSI: J53.1, U$1.PA7, U36.SDA/SDI
- new net IMU_RX: CON65.3, U$1.PA1
- new net IMU_TX: CON65.2, U$1.PA0WKUP
- new net LEDA1: R109.P$1, U$1.PC4
- new net N$257: CON68.5, J52.2
- new net N$258: CON68.4, J53.2
- new net N$259: CON68.3, J54.2
- new net N$260: CON68.2, J55.2
- new net NRST: C211.P$2, CON64.2, U$1.NRST
- new net REGOUT: C196.P$2, U36.REGOUT
- new net SW_CLK: CON64.5, U$1.PA14
- new net SW_DIO: CON64.3, U$1.PA13
- net 3V3: now also C200.P$2, C201.P$2, C202.P$1, C203.P$1, C206.P$1, C207.P$1, C208.P$1, C209.P$1, C210.P$1, C212.P$2, C213.P$2, C214.P$2, C215.P$2, CON64.6, CON68.1, U$1.VBAT, U$1.VDD1, U$1.VDD2, U$1.VDD3, U$1.VDD4, U$1.VDDA, U36.VDD, U36.VDDIO
- net 5V: now also C199.P$2, CON63.VBUS
- net GND: now also C196.P$1, C199.P$1, C200.P$1, C201.P$1, C202.P$2, C203.P$2, C204.P$1, C205.P$1, C206.P$2, C207.P$2, C208.P$2, C209.P$2, C210.P$2, C211.P$1, C212.P$1, C213.P$1, C214.P$1, C215.P$1, CON63.GND, CON63.GND@2, CON64.4, CON65.1, CON68.6, D11.C, U$1.BOOT0, U$1.VSS1, U$1.VSS2, U$1.VSSA; no longer C196.P$2, C199.P$2, CON63.1, CON64.1, R109.P$2, R110.P$2, U39.ADDR, U39.GND, U40.GND
- net N$73: now also D11.A, R109.P$2; no longer C199.P$1, CON63.5, CON64.5, U40.EN, U40.VI
- net N$84: now also C205.P$2, U$1.VCAP1; no longer CON63.2, CON64.2, U36.SDA, U39.SDA
- net N$93: now also C204.P$2, U$1.VCAP2; no longer C196.P$1, U36.VCC, U39.VCCI, U39.VCCP, U40.VO
Other:
- note added: "All in one de chez INVSENSE"
- note added: "L'idee c'etait d'avoir un module IMU deporte (STM32) qui pisse les data de la centrale sur un UART ou de pouvoir l'utiliser en direct avec le SPI sur connecteur."
- note added: "MPU-9250 9DoF"
- note added: "STM32F405_64pins"
- note added: "Use the internal clock ?"
- note added: "Useless ?"
- moved on the sheet: C196, C199, R109
